Commit message: update

File: src/agbot_description/urdf/agbot.urdf.xacro (robot description, xacro)
@@ -10,5 +10,5 @@
     <xacro:property name="velocity" value="10.0" />
     <xacro:property name="scale" value="0.0025 0.0025 0.0025"/>
-    <xacro:property name="wheel_scale" value="0.002 0.002 0.002"/>
+    <xacro:property name="wheel_scale" value="0.006 0.006 0.006"/>
     <!-- Useful Macros -->
     <xacro:macro name="default_inertia" params="mass">
@@ -31,13 +31,13 @@
         </transmission>
     </xacro:macro>
-    <xacro:property name="base_length" value="0.35" />
-    <xacro:property name="base_width" value="0.25" />
-    <xacro:property name="base_height" value="0.10" />
-    <xacro:property name="wheel_radius" value="0.033" />
+    <xacro:property name="base_length" value="1.8288" />
+    <xacro:property name="base_width" value="1.8288" />
+    <xacro:property name="base_height" value="0.762" />
+    <xacro:property name="wheel_radius" value="0.06" />
     <xacro:property name="wheel_length" value="0.05" />
     <xacro:property name="mast_length" value="0.05" />
     <xacro:property name="mast_width" value="0.05" />
     <xacro:property name="mast_height" value="0.01" />
-    <xacro:property name="caster_radius" value="0.035" />
+    <xacro:property name="caster_radius" value="0.06" />
     <link name = "base_footprint" />
     <link name="base_link">
@@ -179,5 +179,5 @@
         <parent link="base_link" />
         <child link="right_wheel_link" />
-        <origin xyz="-${base_length / 4.0} -${(base_width + wheel_length) / 2.0} 0.035" rpy="0 0 0" />
+        <origin xyz="-${base_length / 4.0} -${(base_width + wheel_length) / 2.0} 0.14" rpy="0 0 0" />
         <axis xyz="0 1 0" />
     </joint>
@@ -185,5 +185,5 @@
         <parent link="base_link" />
         <child link="left_wheel_link" />
-        <origin xyz="-${base_length / 4.0} ${(base_width + wheel_length) / 2.0} 0.035" rpy="0 0 0" />
+        <origin xyz="-${base_length / 4.0} ${(base_width + wheel_length) / 2.0} 0.14" rpy="0 0 0" />
         <axis xyz="0 1 0" />
     </joint>
@@ -191,5 +191,5 @@
         <parent link="base_link" />
         <child link="caster_wheel_link" />
-        <origin xyz="${base_length / 3.0} 0 0.008" rpy="0 0 0" />
+        <origin xyz="${base_length / 3.0} 0 0" rpy="0 0 0" />
     </joint>
     <joint name="camera_optical_joint" type="fixed">

File: src/agbot_description/urdf/agbot_arm.xacro (robot description, xacro)
@@ -1,8 +1,8 @@
 <?xml version="1.0"?>
 <robot xmlns:xacro="http://www.ros.org/wiki/xacro" name="agbot_arm">
-    <xacro:property name = "forward_drive_arm_length" value = "1.00" />
+    <xacro:property name = "forward_drive_arm_length" value = "0.75" />
     <xacro:property name = "forward_drive_arm_width" value = "0.05" />
     <xacro:property name = "forward_drive_arm_height" value = "0.005" />
-    <xacro:property name = "horizontal_arm_length" value = "0.740" />
+    <xacro:property name = "horizontal_arm_length" value = "0.555" />
     <xacro:property name = "horizontal_arm_width" value = "0.05" />
     <xacro:property name = "horizontal_arm_height" value = "0.005" />
@@ -18,5 +18,5 @@
     <xacro:property name="effort" value="30.0" />
     <xacro:property name="velocity" value="10.0" />
-    <xacro:property name="arm_scale" value="0.002 0.002 0.002"/>
+    <xacro:property name="arm_scale" value="0.0015 0.0015 0.002"/>
     <xacro:property name="claw_scale" value="0.004 0.004 0.004"/>
     <!-- Useful Macros -->
@@ -44,5 +44,5 @@
         <xacro:default_inertia mass="1.0"/>
         <visual>
-            <origin xyz="-0.1 -0.1 0" rpy="0 0 0"/>
+            <origin xyz="-0.077 -0.075 0" rpy="0 0 0"/>
             <geometry>
                 <mesh filename="file://$(find agbot_description)/meshes/basement.STL" scale="${arm_scale}"/>
@@ -51,5 +51,5 @@
         </visual>
         <collision>
-            <origin xyz="-0.1 -0.1 0" rpy="0 0 0"/>
+            <origin xyz="-0.075 -.075 0" rpy="0 0 0"/>
             <geometry>
                 <mesh filename="file://$(find agbot_description)/meshes/basement.STL" scale="${arm_scale}"/>
@@ -60,5 +60,5 @@
         <xacro:default_inertia mass="0.1"/>
          <visual>
-            <origin xyz="-0.076 -0.0798 -0.121" rpy="0 0 0"/>
+            <origin xyz="-0.059 -0.060 -0.121" rpy="0 0 0"/>
             <geometry>
                 <mesh filename="file://$(find agbot_description)/meshes/base_plate.STL" scale="${arm_scale}"/>
@@ -76,5 +76,5 @@
         <xacro:default_inertia mass="0.1"/>
         <visual>
-            <origin xyz="0.01 -0.006 0.495" rpy="0 ${PI / 2} ${PI / 2}"/>
+            <origin xyz="-0.005 -0.006 0.38" rpy="0 ${PI / 2} ${PI / 2}"/>
             <geometry>
                 <box size="${forward_drive_arm_length} ${forward_drive_arm_width} ${forward_drive_arm_height}" />
@@ -83,5 +83,5 @@
         </visual>
         <collision>
-            <origin xyz="0.01 -0.006 0.495" rpy="0 ${PI / 2} ${PI / 2}"/>
+            <origin xyz="0.01 -0.006 0" rpy="0 ${PI / 2} ${PI / 2}"/>
             <geometry>
                 <box size="${forward_drive_arm_length} ${forward_drive_arm_width} ${forward_drive_arm_height}" />
@@ -109,5 +109,5 @@
         <xacro:default_inertia mass="0.1"/>
         <visual>
-            <origin xyz="0 0 0.37" rpy="0 ${PI / 2} ${PI / 2}"/>
+            <origin xyz="0 0 0.275" rpy="0 ${PI / 2} ${PI / 2}"/>
             <geometry>
                 <box size="${horizontal_arm_length} ${horizontal_arm_width} ${horizontal_arm_height}" />
@@ -116,5 +116,5 @@
         </visual>
         <collision>
-            <origin xyz="0 0 0.37" rpy="0 ${PI / 2} ${PI / 2}"/>
+            <origin xyz="0 0 0.275" rpy="0 ${PI / 2} ${PI / 2}"/>
             <geometry>
                 <box size="${horizontal_arm_length} ${horizontal_arm_width} ${horizontal_arm_height}" />
@@ -222,5 +222,5 @@
         <parent link="base_plate"/>
         <child link="forward_drive_arm"/>
-        <origin xyz="0 0.006 0.07" rpy="-${PI/2} 0 0"/>
+        <origin xyz="0 0 0.066" rpy="-${PI/2} 0 0"/>
         <axis xyz="1 0 0"/>
         <limit lower="0" upper="4.0" effort="${effort}" velocity="${velocity}"/>

File: src/agbot_description/urdf/agbot_full.xacro (robot description, xacro)
@@ -12,5 +12,5 @@
     <xacro:property name="velocity" value="10.0" />
     <xacro:property name="scale" value="0.0025 0.0025 0.0025"/>
-    <xacro:property name="wheel_scale" value="0.002 0.002 0.002"/>
+    <xacro:property name="wheel_scale" value="0.006 0.006 0.006"/>
     <xacro:property name="arm_scale" value="0.002 0.002 0.002"/>
     <xacro:property name="claw_scale" value="0.004 0.004 0.004"/>
@@ -35,7 +35,7 @@
         </transmission>
     </xacro:macro>
-    <xacro:property name="base_length" value="0.35" />
-    <xacro:property name="base_width" value="0.25" />
-    <xacro:property name="base_height" value="0.10" />
+    <xacro:property name="base_length" value="1.8288" />
+    <xacro:property name="base_width" value="1.8288" />
+    <xacro:property name="base_height" value="0.9144" />
     <xacro:property name="wheel_radius" value="0.033" />
     <xacro:property name="wheel_length" value="0.05" />
@@ -50,5 +50,5 @@
     <xacro:property name = "horizontal_arm_width" value = "0.05" />
     <xacro:property name = "horizontal_arm_height" value = "0.005" />
-    <xacro:property name = "cylinder_radius" value = "0.015" />
+    <xacro:property name = "cylinder_radius" value = "0.06" />
     <xacro:property name = "cylinder_length" value = "0.18" />
    <!-- Robot Body -->

File: src/agbot_description/urdf/agbot_full_ros2_control.xacro (robot description, xacro)
@@ -2,65 +2,63 @@
 <robot xmlns:xacro="http://www.ros.org/wiki/xacro" name="agbot">
     <xacro:property name="PI" value="3.14159265359" />
-    <xacro:macro name="RobotSystem" >
-        <ros2_control name="${name}" type="system">
-            <hardware>
-                <plugin>gazebo_ros2_control/GazeboSystem</plugin>
-            </hardware>
-        <!-- BODY -->
-        <joint name="left_wheel_joint">
-            <command_interface name="velocity"/>
-            <state_interface name="position"/>
-            <state_interface name="velocity"/>
-        </joint>
-        <joint name="right_wheel_joint">
-            <command_interface name="velocity"/>
-            <state_interface name="position"/>
-            <state_interface name="velocity"/>
-        </joint>
-        <!-- ARM -->
-        <joint name="arm_base_joint">
-            <command_interface name="position">
-                <param name="min">-${PI}</param>
-                <param name="max">${PI}</param>
-            </command_interface>
-            <state_interface name="position"/>
-        </joint>
-        <joint name="shoulder_joint">
-            <command_interface name="position">
-                <param name="min">0</param>
-                <param name="max">4</param>
-            </command_interface>
-            <state_interface name="position"/>
-        </joint>
-        <joint name="elbow_joint">
-            <command_interface name="position">
-                <param name="min">-${PI}</param>
-                <param name="max">0</param>
-            </command_interface>
-            <state_interface name="position"/>
-        </joint>
-        <joint name="wrist_joint">
-            <command_interface name="position">
-                <param name="min">-${PI/2}</param>
-                <param name="max">${PI/2}</param>
-            </command_interface>
-            <state_interface name="position"/>
-        </joint>
-        <joint name="gripper_right_joint">
-            <command_interface name="position">
-                <param name="min">-${PI/2}</param>
-                <param name="max">0</param>
-            </command_interface>
-            <state_interface name="position"/>
-        </joint>
-        <joint name="gripper_left_joint">
-            <param name="mimic">gripper_right_joint</param>
-            <param name="multiplier">-1</param>
-            <command_interface name="position">
-                <param name="min">0</param>
-                <param name="max">${PI/2}</param>
-            </command_interface>
-        </joint>
-    </ros2_control>
-  </xacro:macro>
+    <ros2_control name="RobotSystem" type="system">
+        <hardware>
+            <plugin>gazebo_ros2_control/GazeboSystem</plugin>
+        </hardware>
+    <!-- BODY -->
+    <joint name="left_wheel_joint">
+        <command_interface name="velocity"/>
+        <state_interface name="position"/>
+        <state_interface name="velocity"/>
+    </joint>
+    <joint name="right_wheel_joint">
+        <command_interface name="velocity"/>
+        <state_interface name="position"/>
+        <state_interface name="velocity"/>
+    </joint>
+    <!-- ARM -->
+    <joint name="arm_base_joint">
+        <command_interface name="position">
+            <param name="min">-${PI}</param>
+            <param name="max">${PI}</param>
+        </command_interface>
+        <state_interface name="position"/>
+    </joint>
+    <joint name="shoulder_joint">
+        <command_interface name="position">
+            <param name="min">0</param>
+            <param name="max">4</param>
+        </command_interface>
+        <state_interface name="position"/>
+    </joint>
+    <joint name="elbow_joint">
+        <command_interface name="position">
+            <param name="min">-${PI}</param>
+            <param name="max">0</param>
+        </command_interface>
+        <state_interface name="position"/>
+    </joint>
+    <joint name="wrist_joint">
+        <command_interface name="position">
+            <param name="min">-${PI/2}</param>
+            <param name="max">${PI/2}</param>
+        </command_interface>
+        <state_interface name="position"/>
+    </joint>
+    <joint name="gripper_right_joint">
+        <command_interface name="position">
+            <param name="min">-${PI/2}</param>
+            <param name="max">0</param>
+        </command_interface>
+        <state_interface name="position"/>
+    </joint>
+    <joint name="gripper_left_joint">
+        <param name="mimic">gripper_right_joint</param>
+        <param name="multiplier">-1</param>
+        <command_interface name="position">
+            <param name="min">0</param>
+            <param name="max">${PI/2}</param>
+        </command_interface>
+    </joint>
+</ros2_control>
 </robot>

File: src/agbot_description/urdf/agbot_ros2_control.xacro (robot description, xacro)
@@ -5,5 +5,4 @@
         <hardware>
           <plugin>gazebo_ros2_control/GazeboSystem</plugin>
-            <!-- <plugin> name="diff_drive_controller" filename="libgazebo_ros_diff_drive.so" </plugin> -->
         </hardware>
         <joint name="left_wheel_joint">

File: src/agbot_description/urdf/common_properties.xacro (robot description, xacro)
@@ -20,4 +20,7 @@
         <color rgba="0.5 0.5 0.5 1.0"/>
     </material>
+    <material name="ClearGrey">
+        <color rgba="0.2 0.2 0.2 0.6"/>
+      </material>
     <material name="orange">
         <color rgba="1.0 0.4235 0.0392 1.0"/>
