Commit message: update

File: src/agbot_full_description/urdf/agbot_full.xacro (robot description, xacro)
@@ -12,6 +12,6 @@
     <xacro:property name="velocity" value="10.0" />
     <xacro:property name="scale" value="0.0025 0.0025 0.0025"/>
-    <xacro:property name="wheel_scale" value="0.002 0.002 0.002"/>
-    <xacro:property name="arm_scale" value="0.002 0.002 0.002"/>
+    <xacro:property name="wheel_scale" value="0.006 0.006 0.006"/>
+    <xacro:property name="arm_scale" value="0.0015 0.0015 0.002"/>
     <xacro:property name="claw_scale" value="0.004 0.004 0.004"/>
     <!-- Useful Macros -->
@@ -35,420 +35,564 @@
         </transmission>
     </xacro:macro>
-    <xacro:property name="base_length" value="0.35" />
-    <xacro:property name="base_width" value="0.25" />
-    <xacro:property name="base_height" value="0.10" />
-    <xacro:property name="wheel_radius" value="0.033" />
+    <xacro:property name="base_length" value="1.8288" />
+    <xacro:property name="base_width" value="1.8288" />
+    <xacro:property name="base_height" value="0.762" />
+    <xacro:property name="wheel_radius" value="0.06" />
     <xacro:property name="wheel_length" value="0.05" />
     <xacro:property name="mast_length" value="0.05" />
     <xacro:property name="mast_width" value="0.05" />
     <xacro:property name="mast_height" value="0.01" />
-    <xacro:property name="caster_radius" value="0.035" />
-    <xacro:property name = "forward_drive_arm_length" value = "1.00" />
+    <xacro:property name="caster_radius" value="0.06" />
+    <xacro:property name = "forward_drive_arm_length" value = "0.75" />
     <xacro:property name = "forward_drive_arm_width" value = "0.05" />
     <xacro:property name = "forward_drive_arm_height" value = "0.005" />
-    <xacro:property name = "horizontal_arm_length" value = "0.740" />
+    <xacro:property name = "horizontal_arm_length" value = "0.555" />
     <xacro:property name = "horizontal_arm_width" value = "0.05" />
     <xacro:property name = "horizontal_arm_height" value = "0.005" />
     <xacro:property name = "cylinder_radius" value = "0.015" />
     <xacro:property name = "cylinder_length" value = "0.18" />
-   <!-- Robot Body -->
-   <link name = "base_footprint" />
-   <link name="base_link">
-      <visual>
-         <geometry>
-               <box size="${base_length} ${base_width} ${base_height}"/>
-         </geometry>
-         <origin xyz="0 0 ${base_height/2}" rpy="0 0 0"/>
-         <material name="maroon"/>
-      </visual>
-      <collision>
-         <geometry>
-               <box size="${base_length*1.1} ${base_width*1.1} ${base_height*1.1}"/>
-         </geometry>
-         <origin xyz="0 0 ${base_height/2}" rpy="0 0 0"/>
-      </collision>
-      <xacro:box_inertia m="10.0" l="${base_length}" w="${base_width}" h="${base_height}"
-                        xyz = "0 0 ${base_height/2}" rpy="0 0 0" />
-   </link>
-   <link name="left_wheel_link" >
-      <visual>
-         <geometry>
-               <mesh filename="file://$(find agbot_full_description)/meshes/left_tire.stl" scale="${wheel_scale}"/>
-               <!-- <cylinder radius = "${wheel_radius}" length = "${wheel_length}" /> -->
-         </geometry>
-         <origin xyz = "0 0 0" rpy = "0 0 0" />
-         <material name = "black" />
-      </visual>
-      <collision>
-               <geometry>
-                  <mesh filename="file://$(find agbot_full_description)/meshes/left_tire.stl" scale="${wheel_scale}"/>
-                  <!-- <cylinder radius = "${wheel_radius}" length = "${wheel_length}" /> -->
-         </geometry>
-         <origin xyz = "0 0 0" rpy = "0 0 0" />
-      </collision>
-      <xacro:wheel_inertia m="1.0" r = "${wheel_radius}" h = "${wheel_length}"
-                              xyz = "0 0 0" rpy = "${Pi/2.0} -${Pi/2.0} 0" />
-   </link>
-   <link name="right_wheel_link" >
-      <visual>
-         <geometry>
-               <mesh filename="file://$(find agbot_full_description)/meshes/right_tire.stl" scale="${wheel_scale}"/>
-               <!-- <cylinder radius = "${wheel_radius}" length = "${wheel_length}" /> -->
-         </geometry>
-         <origin xyz = "0 0 0" rpy = "0 0 0" />
-         <material name = "black" />
-      </visual>
-      <collision>
-         <geometry>
-               <mesh filename="file://$(find agbot_full_description)/meshes/right_tire.stl" scale="${wheel_scale}"/>
-               <!-- <cylinder radius = "${wheel_radius}" length = "${wheel_length}" /> -->
-         </geometry>
-         <origin xyz = "0 0 0" rpy = "0 0 0" />
-      </collision>
-      <xacro:wheel_inertia m="1.0" r = "${wheel_radius}" h = "${wheel_length}"
-                              xyz = "0 0 0" rpy = "${Pi/2.0} -${Pi/2.0} 0" />
-   </link>
-   <link name = "caster_wheel_link">
-      <visual>
-         <geometry>
-               <sphere radius = "${caster_radius}" />
-         </geometry>
-         <origin xyx = "${base_length / 3} 0 ${caster_radius}" rpy = "0 0 0" />
-         <material name = "yellow" />
-      </visual>
-      <collision>
-         <geometry>
-               <sphere radius = "${caster_radius}" />
-         </geometry>
-         <origin xyx = "${base_length / 3} 0 ${caster_radius}" rpy = "0 0 0" />
-      </collision>
-      <xacro:sphere_inertia m = "0.2" r = "${caster_radius}"
-                           xyz = "${base_length / 3} 0 0" rpy = "0 0 0" />
-   </link>
-   <link name="rgb_camera_optical" >
-   </link>
-   <link name="rgb_camera">
-      <xacro:default_inertia mass="0.001"/>
-      <visual>
-         <origin xyz="0 -0.035 0.035" rpy="0 ${Pi/2} 0"/>
-         <geometry>
-               <mesh filename="file://$(find agbot_full_description)/meshes/pi_camera.STL" scale="${scale}"/>
-         </geometry>
-         <material name="grey"/>
-      </visual>
-      <collision>
-         <origin xyz="0.2 0 0" rpy="0 0 0"/>
-         <geometry>
-               <mesh filename="file://$(find agbot_full_description)/meshes/pi_camera.STL" scale="${scale}"/>
-         </geometry>
-      </collision>
-   </link>
-   <link name="mast_link">
-      <visual>
-         <origin xyz="0 0 ${mast_height/2}" rpy="0 0 0"/>
-         <geometry>
-               <box size="${mast_length} ${mast_width} ${mast_height}"/>
-         </geometry>
-         <material name="pink"/>
-      </visual>
-      <collision>
-         <geometry>
-               <box size="${mast_length} ${mast_width} ${mast_height}"/>
-         </geometry>
-         <origin xyz="0 0 0" rpy="0 0 0"/>
-      </collision>
-      <xacro:box_inertia m="0.005" l="${mast_length}" w="${mast_width}" h="${mast_height}"
-                        xyz = "0 0 0" rpy="0 0 0" />
-   </link>
-   <link name="laser_frame">
-   </link>
-   <!-- Robot Arm -->
-   <link name="arm_base_link">
-      <xacro:default_inertia mass="1.0"/>
-      <visual>
-          <origin xyz="-0.1 -0.1 0" rpy="0 0 0"/>
-          <geometry>
-              <mesh filename="file://$(find agbot_full_description)/meshes/basement.STL" scale="${arm_scale}"/>
-          </geometry>
-          <material name="blue"/>
-      </visual>
-      <collision>
-          <origin xyz="-0.1 -0.1 0" rpy="0 0 0"/>
-          <geometry>
-              <mesh filename="file://$(find agbot_full_description)/meshes/basement.STL" scale="${arm_scale}"/>
-          </geometry>
-      </collision>
-  </link>
-  <link name="base_plate">
-      <xacro:default_inertia mass="0.1"/>
-       <visual>
-          <origin xyz="-0.076 -0.0798 -0.121" rpy="0 0 0"/>
-          <geometry>
-              <mesh filename="file://$(find agbot_full_description)/meshes/base_plate.STL" scale="${arm_scale}"/>
-          </geometry>
-          <material name="red"/>
-      </visual>
-      <collision>
-          <origin xyz="-0.076 -0.0798 -0.121" rpy="0 0 0"/>
-          <geometry>
-              <mesh filename="file://$(find agbot_full_description)/meshes/base_plate.STL" scale="${arm_scale}"/>
-          </geometry>
-      </collision>
-  </link>
-  <link name="forward_drive_arm">
-      <xacro:default_inertia mass="0.1"/>
-      <visual>
-          <origin xyz="0.01 -0.006 0.495" rpy="0 ${PI / 2} ${PI / 2}"/>
-          <geometry>
-              <box size="${forward_drive_arm_length} ${forward_drive_arm_width} ${forward_drive_arm_height}" />
-          </geometry>
-          <material name="yellow"/>
-      </visual>
-      <collision>
-          <origin xyz="0.01 -0.006 0.495" rpy="0 ${PI / 2} ${PI / 2}"/>
-          <geometry>
-              <box size="${forward_drive_arm_length} ${forward_drive_arm_width} ${forward_drive_arm_height}" />
-          </geometry>
-      </collision>
-  </link>
-  <link name = "elbow">
-      <visual>
-          <origin xyz="0 0 0" rpy="0 ${PI / 2} 0"/>
-          <geometry>
-              <cylinder length = "${cylinder_length}" radius = "${cylinder_radius}" />
-          </geometry>
-          <material name="white"/>
-      </visual>
-      <collision>
-          <origin xyz="0 0 0" rpy="0 ${PI / 2} 0"/>
-          <geometry>
-              <cylinder length = "${cylinder_length}" radius = "${cylinder_radius}"  />
-          </geometry>
-      </collision>
-      <xacro:cylinder_inertia m = "0.05" r = "${cylinder_radius}" h = "${cylinder_length}"
-                             xyz = "0 0 0" rpy = "0 0 0"/>
-  </link>
-  <link name="horizontal_arm">
-      <xacro:default_inertia mass="0.1"/>
-      <visual>
-          <origin xyz="0 0 0.37" rpy="0 ${PI / 2} ${PI / 2}"/>
-          <geometry>
-              <box size="${horizontal_arm_length} ${horizontal_arm_width} ${horizontal_arm_height}" />
-          </geometry>
-          <material name="green"/>
-      </visual>
-      <collision>
-          <origin xyz="0 0 0.37" rpy="0 ${PI / 2} ${PI / 2}"/>
-          <geometry>
-              <box size="${horizontal_arm_length} ${horizontal_arm_width} ${horizontal_arm_height}" />
-          </geometry>
-      </collision>
-  </link>
-  <link name = "wrist">
-      <visual>
-          <origin xyz="0 0 0" rpy="0 ${PI / 2} 0"/>
-          <geometry>
-              <cylinder length = "${cylinder_length / 2}" radius = "${cylinder_radius}" />
-          </geometry>
-          <material name="white"/>
-      </visual>
-      <collision>
-          <origin xyz="0 0 0" rpy="0 ${PI / 2} 0"/>
-          <geometry>
-              <cylinder length = "${cylinder_length}" radius = "${cylinder_radius}"  />
-          </geometry>
-      </collision>
-      <xacro:cylinder_inertia m = "0.05" r = "${cylinder_radius}" h = "${cylinder_length}"
-                             xyz = "0 0 0" rpy = "0 0 0"/>
-  </link>
-  <link name="claw_support">
-      <xacro:default_inertia mass="0.05"/>
-      <visual>
-          <origin xyz="-${cylinder_length/3.7} 0 0" rpy="0 -${PI/2} -${PI / 2}"/>
-          <geometry>
-              <mesh filename="file://$(find agbot_full_description)/meshes/claw_support.STL" scale="${claw_scale}"/>
-          </geometry>
-          <material name="pink"/>
-      </visual>
-      <collision>
-          <origin xyz="-${cylinder_length/3.7} 0 0" rpy="0 -${PI/2} -${PI / 2}"/>
-          <geometry>
-              <mesh filename="file://$(find agbot_full_description)/meshes/claw_support.STL" scale="${claw_scale}"/>
-          </geometry>
-      </collision>
-  </link>
-  <link name="gripper_right">
-      <xacro:default_inertia mass="0.01"/>
-      <visual>
-          <origin xyz="0.041 0 0.19" rpy="0 ${PI / 2} ${PI / 2}"/>
-          <geometry>
-              <mesh filename="file://$(find agbot_full_description)/meshes/right_finger.STL" scale="${claw_scale}"/>
-          </geometry>
-          <material name="purple"/>
-      </visual>
-      <collision>
-          <origin xyz="0.041 0 0.19" rpy="0 ${PI / 2} ${PI / 2}"/>
-          <geometry>
-              <mesh filename="file://$(find agbot_full_description)/meshes/right_finger.STL" scale="${claw_scale}"/>
-          </geometry>
-      </collision>
-  </link>
-  <link name="gripper_left">
-      <xacro:default_inertia mass="0.01"/>
-      <visual>
-          <origin xyz="0.0147 0 0.19" rpy="0 ${PI / 2} ${PI / 2}"/>
-          <geometry>
-              <mesh filename="file://$(find agbot_full_description)/meshes/left_finger.STL" scale="${claw_scale}"/>
-          </geometry>
-          <material name="purple"/>
-      </visual>
-      <collision>
-          <origin xyz="0.0147 0 0.19" rpy="0 ${PI / 2} ${PI / 2}"/>
-          <geometry>
-              <mesh filename="file://$(find agbot_full_description)/meshes/left_finger.STL" scale="${claw_scale}"/>
-          </geometry>
-      </collision>
-  </link>
-  <link name="arm_rgb_camera_optical" >
-  </link>
-  <link name="arm_rgb_camera">
-      <xacro:default_inertia mass="0.001"/>
-      <visual>
-          <origin xyz="-0.03 -0.055 0.05" rpy="0 ${PI/2} 0"/>
-          <geometry>
-              <mesh filename="file://$(find agbot_full_description)/meshes/pi_camera.STL" scale="${claw_scale}"/>
-          </geometry>
-          <material name="blue"/>
-      </visual>
-      <collision>
-          <origin xyz="0 -.03 0" rpy="0 ${PI/2} 0"/>
-          <geometry>
-              <mesh filename="file://$(find agbot_full_description)/meshes/pi_camera.STL" scale="${claw_scale}"/>
-          </geometry>
-      </collision>
-  </link>
-   <!-- Joint Descriptions -->
-   <!-- Robot Body -->
-   <joint name="base_joint" type="fixed">
-      <parent link="base_footprint" />
-      <child link="base_link" />
-      <origin xyz="0 0 ${wheel_radius}" rpy="0 0 0"/>
-   </joint>
-   <joint name="base_right_wheel_joint" type="continuous">
-      <parent link="base_link" />
-      <child link="right_wheel_link" />
-      <origin xyz="-${base_length / 4.0} -${(base_width + wheel_length) / 2.0} 0.035" rpy="0 0 0" />
-      <axis xyz="0 1 0" />
-   </joint>
-   <joint name="base_left_wheel_joint" type="continuous">
-      <parent link="base_link" />
-      <child link="left_wheel_link" />
-      <origin xyz="-${base_length / 4.0} ${(base_width + wheel_length) / 2.0} 0.035" rpy="0 0 0" />
-      <axis xyz="0 1 0" />
-   </joint>
-   <joint name="base_caster_wheel_joint" type="fixed">
-      <parent link="base_link" />
-      <child link="caster_wheel_link" />
-      <origin xyz="${base_length / 3.0} 0 0.008" rpy="0 0 0" />
-   </joint>
-   <joint name="camera_optical_joint" type="fixed">
-      <parent link="base_link"/>
-      <child link="rgb_camera_optical"/>
-      <origin xyz = "${base_length/2} 0 ${base_height-0.02}" rpy = "0 0 0" />
-   </joint>
-   <joint name = "rgb_camera_joint" type = "fixed" >
-      <parent link = "rgb_camera_optical" />
-      <child link = "rgb_camera" />
-      <origin xyz="0 0 0" rpy="0 0 0"/>
-   </joint>
-   <joint name = "base_mast_joint" type = "fixed">
-      <parent link = "base_link" />
-      <child link = "mast_link" />
-      <origin xyz="${((base_length/2)- 0.05)} 0 ${base_height}" rpy="0 0 0"/>
-   </joint>
-   <joint name="laser_joint" type="fixed">
-      <parent link="mast_link"/>
-      <child link="laser_frame"/>
-      <origin xyz="0 0 ${mast_height + 0.02}" rpy="0 0 0"/>
-   </joint>
+    <xacro:property name = "robo_cylinder_radius" value = "0.2032" />
+    <xacro:property name = "robo_cylinder_length" value = "1.8288" />
+    <xacro:property name = "arm_base_rail_length" value = "1.524" />
+    <xacro:property name = "arm_base_rail_width" value = "0.1524" />
+    <xacro:property name = "arm_base_rail_height" value = "0.0127" />
+    <xacro:property name = "arm_base_car_length" value = "1.524" />
+    <xacro:property name = "arm_base_car_width" value = "0.1524" />
+    <xacro:property name = "arm_base_car_height" value = "0.0127" />
+    <xacro:property name = "box_length" value = "0.3" />
+    <xacro:property name = "box_width" value = "0.1524" />
+    <xacro:property name = "box_height" value = "0.0762" />
+    <!-- Robot Body -->
+    <link name = "base_footprint" />
+    <link name="base_link">
+        <visual>
+            <geometry>
+                <box size="${base_length} ${base_width} ${base_height}"/>
+            </geometry>
+            <origin xyz="0 0 ${base_height/2}" rpy="0 0 0"/>
+            <material name="maroon"/>
+        </visual>
+        <collision>
+            <geometry>
+                <box size="${base_length*1.1} ${base_width*1.1} ${base_height*1.1}"/>
+            </geometry>
+            <origin xyz="0 0 ${base_height/2}" rpy="0 0 0"/>
+        </collision>
+        <xacro:box_inertia m="18.0" l="${base_length}" w="${base_width}" h="${base_height}"
+                           xyz = "0 0 ${base_height/2}" rpy="0 0 0" />
+    </link>
+    <link name="left_wheel_link" >
+        <visual>
+            <geometry>
+                <mesh filename="file://$(find agbot_full_description)/meshes/left_tire.stl" scale="${wheel_scale}"/>
+            </geometry>
+            <origin xyz = "0 0 0" rpy = "0 0 0" />
+            <material name = "black" />
+        </visual>
+        <collision>
+                <geometry>
+                    <mesh filename="file://$(find agbot_full_description)/meshes/left_tire.stl" scale="${wheel_scale}"/>
+            </geometry>
+            <origin xyz = "0 0 0" rpy = "0 0 0" />
+        </collision>
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
File: src/agbot_full_description/urdf/agbot_full_common_properties.xacro (robot description, xacro)
@@ -20,4 +20,7 @@
         <color rgba="0.5 0.5 0.5 1.0"/>
     </material>
+    <material name="ClearGrey">
+        <color rgba="0.2 0.2 0.2 0.75"/>
+      </material>
     <material name="orange">
         <color rgba="1.0 0.4235 0.0392 1.0"/>

File: src/agbot_full_description/urdf/agbot_full_gazebo.xacro (robot description, xacro)
@@ -1,4 +1,4 @@
 <?xml version="1.0" encoding="utf-8"?>
-<robot xmlns:xacro="http://www.ros.org/wiki/xacro" name="agbot">
+<robot xmlns:xacro="http://www.ros.org/wiki/xacro" name="agbot_full">
     <!-- Gazebo ros2_control plugin -->
     <gazebo>
@@ -8,5 +8,5 @@
             <parameters>$(find agbot_full_controller)/config/agbot_full_controllers.yaml</parameters>
             <controller_manager_prefix_node_name>controller_manager</controller_manager_prefix_node_name>
-            <update_rate>50</update_rate>
+            <update_rate>100</update_rate>
             <left_joint>base_left_wheel_joint</left_joint>
             <right_joint>base_right_wheel_joint</right_joint>
@@ -66,6 +66,6 @@
               </image>
               <clip>
-                  <near>0.05</near>
-                  <far>10.0</far>
+                  <near>0.01</near>
+                  <far>6.0</far>
               </clip>
           </camera>
@@ -124,4 +124,10 @@
      </gazebo>
     <!-- Robot Arm -->
+    <gazebo reference="arm_base_rail_link">
+        <material>Gazebo/White</material>
+    </gazebo>
+    <gazebo reference="arm_base_car_link">
+        <material>Gazebo/Black</material>
+    </gazebo>
      <gazebo reference="arm_base_link">
         <material>Gazebo/Blue</material>

File: src/agbot_full_description/urdf/agbot_full_ros2_control.xacro (robot description, xacro)
@@ -1,17 +1,18 @@
 <?xml version="1.0" encoding="utf-8"?>
-<robot xmlns:xacro="http://www.ros.org/wiki/xacro" name="agbot">
+<robot xmlns:xacro="http://www.ros.org/wiki/xacro" name="agbot_full">
     <xacro:property name="PI" value="3.14159265359" />
-    <xacro:macro name="RobotSystem" >
-        <ros2_control name="${name}" type="system">
-            <hardware>
-                <plugin>gazebo_ros2_control/GazeboSystem</plugin>
-            </hardware>
+    <xacro:property name = "arm_base_rail_length" value = "1.524" />
+    <xacro:property name = "arm_base_car_length" value = "0.1524" />
+    <ros2_control name="RobotSystem" type="system">
+        <hardware>
+            <plugin>gazebo_ros2_control/GazeboSystem</plugin>
+        </hardware>
         <!-- BODY -->
-        <joint name="left_wheel_joint">
+        <joint name="base_left_wheel_joint">
             <command_interface name="velocity"/>
             <state_interface name="position"/>
             <state_interface name="velocity"/>
         </joint>
-        <joint name="right_wheel_joint">
+        <joint name="base_right_wheel_joint">
             <command_interface name="velocity"/>
             <state_interface name="position"/>
@@ -19,4 +20,18 @@
         </joint>
         <!-- ARM -->
+        <joint name="arm_base_to_arm_car_joint">
+            <command_interface name="position">
+                <param name="min">0</param>
+                <param name="max">${(arm_base_rail_length / 2) + (arm_base_rail_length / 4)}</param>
+            </command_interface>
+            <state_interface name="position"/>
+        </joint>
+        <joint name="mid_rail_joint">
+            <command_interface name="position">
+                <param name="min">-${arm_base_rail_length/4}</param>
+                <param name="max">${((arm_base_rail_length / 2) + (arm_base_rail_length / 4))/2}</param>
+            </command_interface>
+            <state_interface name="position"/>
+        </joint>
         <joint name="arm_base_joint">
             <command_interface name="position">
@@ -63,4 +78,3 @@
         </joint>
     </ros2_control>
-  </xacro:macro>
 </robot>
