Commit message: Update on 06SEP2024

File: src/agbot_description/urdf/agbot_arm.xacro (robot description, xacro)
@@ -222,5 +222,5 @@
         <parent link="base_plate"/>
         <child link="forward_drive_arm"/>
-        <origin xyz="0 0 0.066" rpy="-${PI/2} 0 0"/>
+        <origin xyz="0 0 .075" rpy="-${PI/2} 0 0"/>
         <axis xyz="1 0 0"/>
         <limit lower="0" upper="4.0" effort="${effort}" velocity="${velocity}"/>

File: src/agbot_description/urdf/agbot_arm_extender.xacro (robot description, xacro)
@@ -33,4 +33,5 @@
     <xacro:property name="arm_scale" value="0.0015 0.0015 0.002"/>
     <xacro:property name="claw_scale" value="0.004 0.004 0.004"/>
+    <xacro:property name="claw_camera_scale" value="0.002 0.002 0.002"/>
     <!-- Useful Macros -->
     <xacro:macro name="default_inertia" params="mass">
@@ -148,54 +149,45 @@
         <collision>
             <geometry>
+                <box size="${arm_base_rail_length} ${arm_base_rail_width} ${arm_base_rail_height}"/>
+            </geometry>
+            <origin xyz="0 0 0" rpy="0 0 0"/>
+        </collision>
+        <xacro:box_inertia m="2.0" l="${arm_base_rail_length}" w="${arm_base_rail_width}" h="${arm_base_rail_height}"
+                        xyz = "0 0 ${arm_base_rail_height/2}" rpy="0 0 0" />
+    </link>
+    <link name="arm_mid_rail_link">
+        <visual>
+            <geometry>
+                <box size="${arm_base_rail_length} ${arm_base_rail_width} ${arm_base_rail_height}"/>
+            </geometry>
+            <origin xyz="0 0 0" rpy="0 0 0"/>
+            <material name="black"/>
+        </visual>
+        <collision>
+            <geometry>
                  <box size="${arm_base_rail_length} ${arm_base_rail_width} ${arm_base_rail_height}"/>
             </geometry>
-            <origin xyz="${arm_base_rail_length/2} ${arm_base_rail_width/2} ${arm_base_rail_height/2}" rpy="0 0 0"/>
+            <origin xyz="0 0 0" rpy="0 0 0"/>
         </collision>
         <xacro:box_inertia m="2.0" l="${arm_base_rail_length}" w="${arm_base_rail_width}" h="${arm_base_rail_height}"
                            xyz = "0 0 ${arm_base_rail_height/2}" rpy="0 0 0" />
     </link>
-    <gazebo reference="arm_base_rail_link">
-        <material>Gazebo/White</material>
-    </gazebo>
-    <link name="arm_mid_rail_link">
-        <visual>
-            <geometry>
-                <box size="${arm_base_rail_length} ${arm_base_rail_width} ${arm_base_rail_height}"/>
-            </geometry>
-            <origin xyz="0 0 0" rpy="0 0 0"/>
+    <link name="arm_base_car_link">
+        <visual>
+            <geometry>
+                <box size="${arm_base_car_length} ${arm_base_car_width} ${arm_base_car_height}"/>
+            </geometry>
+            <origin xyz="0 0 ${arm_base_car_height/2}" rpy="0 0 0"/>
             <material name="white"/>
         </visual>
         <collision>
             <geometry>
-                 <box size="${arm_base_rail_length} ${arm_base_rail_width} ${arm_base_rail_height}"/>
-            </geometry>
-            <origin xyz="${arm_base_rail_length/2} ${arm_base_rail_width/2} ${arm_base_rail_height/2}" rpy="0 0 0"/>
-        </collision>
-        <xacro:box_inertia m="2.0" l="${arm_base_rail_length}" w="${arm_base_rail_width}" h="${arm_base_rail_height}"
-                           xyz = "0 0 ${arm_base_rail_height/2}" rpy="0 0 0" />
-    </link>
-    <gazebo reference="arm_mid_rail_link">
-        <material>Gazebo/White</material>
-    </gazebo>
-    <link name="arm_base_car_link">
-        <visual>
-            <geometry>
                 <box size="${arm_base_car_length} ${arm_base_car_width} ${arm_base_car_height}"/>
             </geometry>
             <origin xyz="0 0 ${arm_base_car_height/2}" rpy="0 0 0"/>
-            <material name="black"/>
-        </visual>
-        <collision>
-            <geometry>
-                 <box size="${arm_base_car_length} ${arm_base_car_width} ${arm_base_car_height}"/>
-            </geometry>
-            <origin xyz="${arm_base_car_length/2} ${arm_base_car_width/2} ${arm_base_car_height/2}" rpy="0 0 0"/>
         </collision>
         <xacro:box_inertia m="2.0" l="${arm_base_car_length}" w="${arm_base_car_width}" h="${arm_base_car_height}"
                            xyz = "0 0 ${arm_base_car_height/2}" rpy="0 0 0" />
     </link>
-    <gazebo reference="arm_base_car_link">
-        <material>Gazebo/Black</material>
-    </gazebo>
     <link name="arm_base_link">
         <xacro:default_inertia mass="1.0"/>
@@ -349,14 +341,14 @@
         <xacro:default_inertia mass="0.001"/>
         <visual>
-            <origin xyz="-0.03 -0.055 0.05" rpy="0 ${PI/2} 0"/>
-            <geometry>
-                <mesh filename="file://$(find agbot_description)/meshes/pi_camera.STL" scale="${claw_scale}"/>
+            <origin xyz="-0.03 -0.028 0.025" rpy="0 ${PI/2} 0"/>
+            <geometry>
+                <mesh filename="file://$(find agbot_description)/meshes/pi_camera.STL" scale="${claw_camera_scale}"/>
             </geometry>
             <material name="blue"/>
         </visual>
         <collision>
-            <origin xyz="0 -.03 0" rpy="0 ${PI/2} 0"/>
-            <geometry>
-                <mesh filename="file://$(find agbot_description)/meshes/pi_camera.STL" scale="${claw_scale}"/>
+            <origin xyz="-0.03 -0.028 0.025" rpy="0 ${PI/2} 0"/>
+            <geometry>
+                <mesh filename="file://$(find agbot_description)/meshes/pi_camera.STL" scale="${claw_camera_scale}"/>
             </geometry>
         </collision>
@@ -468,10 +460,10 @@
         <parent link="claw_support"/>
         <child link="arm_rgb_camera_optical"/>
-        <origin xyz = "0 .13 0.085" rpy = "0 0 0" />
+        <origin xyz = "0 .10 0.085" rpy = "0 0 0" />
     </joint>
     <joint name = "arm_rgb_camera_joint" type = "fixed" >
         <parent link = "arm_rgb_camera_optical" />
         <child link = "arm_rgb_camera" />
-        <origin xyz="0 0 0.015" rpy="0 -${PI/2} 0"/>
+        <origin xyz="0 0 0.03" rpy="0 -${PI/2} 0"/>
     </joint>
     <xacro:default_transmission name="arm_base_to_arm_car_joint" />

File: src/agbot_description/urdf/agbot_arm_extender_gazebo.xacro (robot description, xacro)
@@ -33,4 +33,13 @@
     </sensor>
   </gazebo>
+  <gazebo reference="arm_base_rail_link">
+    <material>Gazebo/White</material>
+  </gazebo>
+  <gazebo reference="arm_mid_rail_link">
+      <material>Gazebo/Black</material>
+  </gazebo>
+  <gazebo reference="arm_base_car_link">
+      <material>Gazebo/White</material>
+  </gazebo>
   <gazebo reference="arm_base_link">
     <material>Gazebo/Blue</material>

File: src/agbot_description/urdf/agbot_full.xacro (robot description, xacro)
@@ -163,10 +163,4 @@
    <link name="laser_frame">
    </link>
-    <!-- Transition Joint  -->
-    <joint name = "body_arm_joint" type = "fixed">
-      <parent link = "base_link"/>
-      <child link = "arm_base_link" />
-      <origin xyz = "${base_length/3} 0 ${base_height}" rpy = "0 0 0" />
-   </joint>
    <!-- Robot Arm -->
    <link name="arm_base_link">
@@ -378,10 +372,16 @@
       <origin xyz="0 0 ${mast_height + 0.02}" rpy="0 0 0"/>
    </joint>
+    <!-- Transition Joint  -->
+    <joint name = "body_arm_joint" type = "fixed">
+        <parent link = "base_link"/>
+        <child link = "arm_base_link" />
+        <origin xyz = "${base_length/3} 0 ${base_height}" rpy = "0 0 0" />
+     </joint>
    <!-- Robot Arm -->
-   <joint name="virtual_joint" type="fixed">
+   <!-- <joint name="virtual_joint" type="fixed">
       <parent link="world"/>
       <child link="arm_base_link"/>
       <origin xyz="0 0 0" rpy="0 0 0"/>
-   </joint>
+   </joint>  -->
    <joint name ="arm_base_joint" type="revolute">
          <parent link="arm_base_link"/>

File: src/agbot_full_description/urdf/agbot_full.xacro (robot description, xacro)
@@ -12,7 +12,36 @@
     <xacro:property name="velocity" value="10.0" />
     <xacro:property name="scale" value="0.0025 0.0025 0.0025"/>
-    <xacro:property name="wheel_scale" value="0.006 0.006 0.006"/>
+    <xacro:property name="wheel_scale" value="0.01 0.01 0.01"/>
     <xacro:property name="arm_scale" value="0.0015 0.0015 0.002"/>
     <xacro:property name="claw_scale" value="0.004 0.004 0.004"/>
+    <xacro:property name="claw_camera_scale" value="0.002 0.002 0.002"/>
+    <xacro:property name="base_length" value="1.8288" />
+    <xacro:property name="base_width" value="1.8288" />
+    <xacro:property name="base_height" value="0.762" />
+    <xacro:property name="wheel_radius" value="0.162" />
+    <xacro:property name="wheel_length" value="0.05" />
+    <xacro:property name="mast_length" value="0.05" />
+    <xacro:property name="mast_width" value="0.05" />
+    <xacro:property name="mast_height" value="0.03" />
+    <xacro:property name="caster_radius" value="0.162" />
+    <xacro:property name = "forward_drive_arm_length" value = "0.75" />
+    <xacro:property name = "forward_drive_arm_width" value = "0.05" />
+    <xacro:property name = "forward_drive_arm_height" value = "0.005" />
+    <xacro:property name = "horizontal_arm_length" value = "0.555" />
+    <xacro:property name = "horizontal_arm_width" value = "0.05" />
+    <xacro:property name = "horizontal_arm_height" value = "0.005" />
+    <xacro:property name = "cylinder_radius" value = "0.015" />
+    <xacro:property name = "cylinder_length" value = "0.18" />
+    <xacro:property name = "robo_cylinder_radius" value = "0.2032" />
+    <xacro:property name = "robo_cylinder_length" value = "1.8288" />
+    <xacro:property name = "arm_base_rail_length" value = "1.524" />
+    <xacro:property name = "arm_base_rail_width" value = "0.1524" />
+    <xacro:property name = "arm_base_rail_height" value = "0.0127" />
+    <xacro:property name = "arm_base_car_length" value = "1.524" />
+    <xacro:property name = "arm_base_car_width" value = "0.1524" />
+    <xacro:property name = "arm_base_car_height" value = "0.0127" />
+    <xacro:property name = "box_length" value = "0.28" />
+    <xacro:property name = "box_width" value = "0.1524" />
+    <xacro:property name = "box_height" value = "0.0762" />
     <!-- Useful Macros -->
     <xacro:macro name="default_inertia" params="mass">
@@ -35,34 +64,20 @@
         </transmission>
     </xacro:macro>
-    <xacro:property name="base_length" value="1.8288" />
-    <xacro:property name="base_width" value="1.8288" />
-    <xacro:property name="base_height" value="0.762" />
-    <xacro:property name="wheel_radius" value="0.06" />
-    <xacro:property name="wheel_length" value="0.05" />
-    <xacro:property name="mast_length" value="0.05" />
-    <xacro:property name="mast_width" value="0.05" />
-    <xacro:property name="mast_height" value="0.01" />
-    <xacro:property name="caster_radius" value="0.06" />
-    <xacro:property name = "forward_drive_arm_length" value = "0.75" />
-    <xacro:property name = "forward_drive_arm_width" value = "0.05" />
-    <xacro:property name = "forward_drive_arm_height" value = "0.005" />
-    <xacro:property name = "horizontal_arm_length" value = "0.555" />
-    <xacro:property name = "horizontal_arm_width" value = "0.05" />
-    <xacro:property name = "horizontal_arm_height" value = "0.005" />
-    <xacro:property name = "cylinder_radius" value = "0.015" />
-    <xacro:property name = "cylinder_length" value = "0.18" />
-    <xacro:property name = "robo_cylinder_radius" value = "0.2032" />
-    <xacro:property name = "robo_cylinder_length" value = "1.8288" />
-    <xacro:property name = "arm_base_rail_length" value = "1.524" />
-    <xacro:property name = "arm_base_rail_width" value = "0.1524" />
-    <xacro:property name = "arm_base_rail_height" value = "0.0127" />
-    <xacro:property name = "arm_base_car_length" value = "1.524" />
-    <xacro:property name = "arm_base_car_width" value = "0.1524" />
-    <xacro:property name = "arm_base_car_height" value = "0.0127" />
-    <xacro:property name = "box_length" value = "0.3" />
-    <xacro:property name = "box_width" value = "0.1524" />
-    <xacro:property name = "box_height" value = "0.0762" />
+    <xacro:macro name="prismatic_transmission" params="name">
+        <transmission name="${name}_prismatic_transmission">
+            <type>transmission_interface/SimpleTransmission</type>
+            <!-- <plugin>hardware_interface/VelocityJointInterface</plugin> -->
+            <joint name="${name}">
+                <hardwareInterface>hardware_interface/PositionJointInterface</hardwareInterface>
+            </joint>
+            <actuator name="${name}_motor">
+                <hardwareInterface>hardware_interface/PositionJointInterface</hardwareInterface>
+                <mechanicalReduction>1</mechanicalReduction>
+            </actuator>
+        </transmission>
+    </xacro:macro>
     <!-- Robot Body -->
-    <link name = "base_footprint" />
+    <link name = "base_footprint">
+    </link>
     <link name="base_link">
         <visual>
@@ -204,5 +219,5 @@
         <collision>
             <geometry>
-                <cylinder length = "${robo_cylinder_radius}" radius = "${robo_cylinder_length}" />
+                <cylinder length = "${robo_cylinder_length}" radius = "${robo_cylinder_radius}" />
             </geometry>
             <origin xyz = "0 0 0" rpy = "0 0 0" />
@@ -223,5 +238,5 @@
                 <box size="${arm_base_rail_length} ${arm_base_rail_width} ${arm_base_rail_height}"/>
             </geometry>
-            <origin xyz="${arm_base_rail_length/2} ${arm_base_rail_width/2} ${arm_base_rail_height/2}" rpy="0 0 0"/>
+            <origin xyz="0 0 0" rpy="0 0 0"/>
         </collision>
         <xacro:box_inertia m="2.0" l="${arm_base_rail_length}" w="${arm_base_rail_width}" h="${arm_base_rail_height}"
@@ -234,5 +249,5 @@
             </geometry>
             <origin xyz="0 0 0" rpy="0 0 0"/>
-            <material name="white"/>
+            <material name="black"/>
         </visual>
         <collision>
@@ -240,12 +255,9 @@
                  <box size="${arm_base_rail_length} ${arm_base_rail_width} ${arm_base_rail_height}"/>
             </geometry>
-            <origin xyz="${arm_base_rail_length/2} ${arm_base_rail_width/2} ${arm_base_rail_height/2}" rpy="0 0 0"/>
+            <origin xyz="0 0 0" rpy="0 0 0"/>
         </collision>
         <xacro:box_inertia m="2.0" l="${arm_base_rail_length}" w="${arm_base_rail_width}" h="${arm_base_rail_height}"
                            xyz = "0 0 ${arm_base_rail_height/2}" rpy="0 0 0" />
     </link>
-    <gazebo reference="arm_mid_rail_link">
-        <material>Gazebo/White</material>
-    </gazebo>
     <link name="arm_base_car_link">
         <visual>
@@ -254,5 +266,5 @@
             </geometry>
             <origin xyz="0 0 ${arm_base_car_height/2}" rpy="0 0 0"/>
-            <material name="black"/>
+            <material name="white"/>
         </visual>
         <collision>
@@ -260,5 +272,5 @@
                 <box size="${arm_base_car_length} ${arm_base_car_width} ${arm_base_car_height}"/>
             </geometry>
-            <origin xyz="${arm_base_car_length/2} ${arm_base_car_width/2} ${arm_base_car_height/2}" rpy="0 0 0"/>
+            <origin xyz="0 0 ${arm_base_car_height/2}" rpy="0 0 0"/>
         </collision>
         <xacro:box_inertia m="2.0" l="${arm_base_car_length}" w="${arm_base_car_width}" h="${arm_base_car_height}"
@@ -307,5 +319,5 @@
         </visual>
         <collision>
-            <origin xyz="0.01 -0.006 0" rpy="0 ${PI / 2} ${PI / 2}"/>
+            <origin xyz="0.01 -0.006 0.38" rpy="0 ${PI / 2} ${PI / 2}"/>
             <geometry>
                 <box size="${forward_drive_arm_length} ${forward_drive_arm_width} ${forward_drive_arm_height}" />
@@ -416,14 +428,14 @@
         <xacro:default_inertia mass="0.001"/>
         <visual>
-            <origin xyz="-0.03 -0.055 0.05" rpy="0 ${PI/2} 0"/>
-            <geometry>
-                <mesh filename="file://$(find agbot_full_description)/meshes/pi_camera.STL" scale="${claw_scale}"/>
+            <origin xyz="-0.03 -0.028 0.025" rpy="0 ${PI/2} 0"/>
+            <geometry>
+                <mesh filename="file://$(find agbot_full_description)/meshes/pi_camera.STL" scale="${claw_camera_scale}"/>
             </geometry>
             <material name="blue"/>
         </visual>
         <collision>
-            <origin xyz="0 -.03 0" rpy="0 ${PI/2} 0"/>
-            <geometry>
-                <mesh filename="file://$(find agbot_full_description)/meshes/pi_camera.STL" scale="${claw_scale}"/>
+            <origin xyz="-0.03 -0.028 0.025" rpy="0 ${PI/2} 0"/>
+            <geometry>
+                <mesh filename="file://$(find agbot_full_description)/meshes/pi_camera.STL" scale="${claw_camera_scale}"/>
             </geometry>
         </collision>
@@ -439,5 +451,5 @@
         <parent link="base_link" />
         <child link="right_wheel_link" />
-        <origin xyz="-${base_length / 4.0} -${(base_width + wheel_length) / 2.0} 0.14" rpy="0 0 0" />
+        <origin xyz="-${base_length / 4.0} -${(base_width + wheel_length) / 2.0} ${wheel_radius}" rpy="0 0 0" />
         <axis xyz="0 1 0" />
     </joint>
@@ -445,5 +457,5 @@
         <parent link="base_link" />
         <child link="left_wheel_link" />
-        <origin xyz="-${base_length / 4.0} ${(base_width + wheel_length) / 2.0} 0.14" rpy="0 0 0" />
+        <origin xyz="-${base_length / 4.0} ${(base_width + wheel_length) / 2.0} ${wheel_radius}" rpy="0 0 0" />
         <axis xyz="0 1 0" />
     </joint>
@@ -456,5 +468,5 @@
         <parent link="base_link"/>
         <child link="rgb_camera_optical"/>
-        <origin xyz = "${base_length/2} 0 ${base_height-0.02}" rpy = "0 0 0" />
+        <origin xyz = "${base_length/2} 0 ${base_height-(base_height/10)}" rpy = "0 0 0" />
     </joint>
     <joint name = "rgb_camera_joint" type = "fixed" >
@@ -466,10 +478,10 @@
         <parent link = "base_link" />
         <child link = "mast_link" />
-        <origin xyz="${((base_length/2)- 0.05)} 0 ${base_height}" rpy="0 0 0"/>
+        <origin xyz="${((base_length / 2) + (mast_length / 2))} 0 ${3 * base_height / 4}" rpy="0 0 0"/>
     </joint>
     <joint name="laser_joint" type="fixed">
         <parent link="mast_link"/>
         <child link="laser_frame"/>
-        <origin xyz="0 0 ${mast_height + 0.02}" rpy="0 0 0"/>
+        <origin xyz="0 0 0" rpy="0 0 0"/>
     </joint>
     <!-- Transition Joint  -->
@@ -484,9 +496,9 @@
         <origin xyz = "0 0 ${base_height + (3*arm_base_rail_height)}" rpy = "0 0 ${PI/2}" />
      </joint>
-     <joint name = "mid_rail_joint" type = "prismatic">
+     <joint name = "base_rail_to_ mid_rail_joint" type = "prismatic">
         <parent link = "arm_base_rail_link"/>
         <child link="arm_mid_rail_link" />
         <origin xyz = "0 0 ${arm_base_rail_height}" rpy = "0 0 0" />
-        <limit effort="100.0" lower="0" upper="${((arm_base_rail_length / 2) + (arm_base_rail_length / 4))/2}" velocity="0.5"/>
+        <limit lower="0" upper="${((arm_base_rail_length / 2) + (arm_base_rail_length / 4))/2}" effort="100.0" velocity="0.5"/>
      </joint>
      <joint name = "box_one_joint" type = "fixed">
@@ -511,9 +523,9 @@
      </joint>
     <!-- Robot Arm -->
-    <joint name = "arm_base_to_arm_car_joint" type = "prismatic">
+    <joint name = "mid_rail_to_arm_car_joint" type = "prismatic">
         <parent link = "arm_mid_rail_link"/>
         <child link = "arm_base_car_link"/>
         <origin xyz = "0 0 ${arm_base_rail_height}" rpy = "0 0 0"/>
-        <limit effort="100.0" lower="0" upper="${(arm_base_rail_length / 2) + (arm_base_rail_length / 4)}" velocity="0.5"/>
+        <limit lower="0" upper="${(arm_base_rail_length / 2) + (arm_base_rail_length / 4)}" effort="100.0" velocity="0.5"/>
     </joint>
     <joint name = "arm_car_to_arm_base_joint" type = "fixed">
@@ -533,5 +545,5 @@
         <parent link="base_plate"/>
         <child link="forward_drive_arm"/>
-        <origin xyz="0 0 0.066" rpy="-${PI/2} 0 0"/>
+        <origin xyz="0 0 0.075" rpy="-${PI/2} 0 0"/>
         <axis xyz="1 0 0"/>
         <limit lower="0" upper="4.0" effort="${effort}" velocity="${velocity}"/>
@@ -564,5 +576,5 @@
         <parent link="claw_support"/>
         <child link="gripper_right"/>
-        <origin xyz="-0.033 -0.012 0.083"/>
+        <origin xyz="-0.035 -0.014 0.083"/>
         <axis xyz="0 1 0"/>
         <limit lower="-${PI / 2}" upper="0.0" effort="${effort}" velocity="${velocity}"/>
@@ -572,5 +584,5 @@
         <parent link="claw_support"/>
         <child link="gripper_left"/>
-        <origin xyz="0.038 -0.012 0.083"/>
+        <origin xyz="0.040 -0.014 0.083"/>
         <axis xyz="0 1 0"/>
         <limit lower="0.0" upper="${PI / 2}" effort="${effort}" velocity="${velocity}"/>
@@ -579,10 +591,10 @@
         <parent link="claw_support"/>
         <child link="arm_rgb_camera_optical"/>
-        <origin xyz = "0 .07 0.09" rpy = "0 0 0" />
+        <origin xyz = "0 .10 0.085" rpy = "0 0 0" />
     </joint>
     <joint name = "arm_rgb_camera_joint" type = "fixed" >
         <parent link = "arm_rgb_camera_optical" />
         <child link = "arm_rgb_camera" />
-        <origin xyz="0 0 0.015" rpy="0 -${PI/2} 0"/>
+        <origin xyz="0 0 0.03" rpy="0 -${PI/2} 0"/>
     </joint>
     <!-- Robot Body -->
@@ -590,5 +602,6 @@
     <xacro:default_transmission name="base_left_wheel_joint" />
     <!-- Robot Arm -->
-    <xacro:default_transmission name="arm_base_to_arm_car_joint" />
+    <xacro:prismatic_transmission name = "mid_rail_joint" />
+    <xacro:prismatic_transmission name="arm_base_to_arm_car_joint" />
     <xacro:default_transmission name="arm_base_joint" />
     <xacro:default_transmission name="shoulder_joint" />

File: src/agbot_full_description/urdf/agbot_full_gazebo.xacro (robot description, xacro)
@@ -108,7 +108,11 @@
      <gazebo reference="left_wheel_link">
         <material>Gazebo/Black</material>
+        <mu1 value="0.8"/>
+        <mu2 value="0.8"/>
      </gazebo>
      <gazebo reference="right_wheel_link">
         <material>Gazebo/Black</material>
+        <mu1 value="0.8"/>
+        <mu2 value="0.8"/>
      </gazebo>
      <gazebo reference="caster_wheel_link">
@@ -127,6 +131,21 @@
         <material>Gazebo/White</material>
     </gazebo>
+    <gazebo reference="arm_mid_rail_link">
+        <material>Gazebo/Black</material>
+        <kp>1000000.0</kp>
+        <kd>100.0</kd>
+        <mu1>30.0</mu1>
+        <mu2>30.0</mu2>
+        <maxVel>0.5</maxVel>
+        <minDepth>0.001</minDepth>
+    </gazebo>
     <gazebo reference="arm_base_car_link">
-        <material>Gazebo/Black</material>
+        <material>Gazebo/White</material>
+        <kp>1000000.0</kp>
+        <kd>100.0</kd>
+        <mu1>30.0</mu1>
+        <mu2>30.0</mu2>
+        <maxVel>0.5</maxVel>
+        <minDepth>0.001</minDepth>
     </gazebo>
      <gazebo reference="arm_base_link">
