Commit message: Update on 06SEP2024

File: src/agbot_full_description/urdf/agbot_full_ros2_control.xacro (robot description, xacro)
@@ -20,17 +20,21 @@
         </joint>
         <!-- ARM -->
-        <joint name="arm_base_to_arm_car_joint">
+        <joint name="base_rail_to_ mid_rail_joint">
             <command_interface name="position">
                 <param name="min">0</param>
-                <param name="max">${(arm_base_rail_length / 2) + (arm_base_rail_length / 4)}</param>
-            </command_interface>
-            <state_interface name="position"/>
-        </joint>
-        <joint name="mid_rail_joint">
-            <command_interface name="position">
-                <param name="min">-${arm_base_rail_length/4}</param>
                 <param name="max">${((arm_base_rail_length / 2) + (arm_base_rail_length / 4))/2}</param>
             </command_interface>
             <state_interface name="position"/>
+            <state_interface name="velocity"/>
+            <state_interface name="effort"/>
+        </joint>
+        <joint name="mid_rail_to_arm_car_joint">
+            <command_interface name="position">
+                <param name="min">0</param>
+                <param name="max">$${(arm_base_rail_length / 2) + (arm_base_rail_length / 4)}</param>
+            </command_interface>
+            <state_interface name="position"/>
+            <state_interface name="velocity"/>
+            <state_interface name="effort"/>
         </joint>
         <joint name="arm_base_joint">
