Commit message: Cleanup Update

File: install/agbot_full_description/share/agbot_full_description/urdf/agbot_full.urdf (robot description, URDF)
Before this commit: robot agbot_full, 28 links, 27 joints
Links:
- removed link arm_rgb_camera
- removed link arm_rgb_camera_optical
- removed link base_plate
- removed link claw_support
- removed link elbow
- removed link forward_drive_arm
- removed link gripper_left
- removed link gripper_right
- removed link horizontal_arm
- removed link roboball_cylinder
- removed link wrist
- added link arm_rgb_camera_link, mass 0.001; collision mesh filename=file:///home/albert/rad_ws/install/agbot_full_description/s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 scale=0.002 0.002 0.002; visual mesh filename=file:///home/albert/rad_ws/install/agbot_full_description/s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 scale=0.002 0.002 0.002
- added link arm_rgb_camera_optical_link
- added link base_plate_link, mass 0.1; collision mesh filename=file:///home/albert/bcdc_ws/install/agbot_description/share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 scale=0.0015 0.0015 0.002; visual mesh filename=file:///home/albert/bcdc_ws/install/agbot_description/share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 scale=0.0015 0.0015 0.002
- added link claw_support_link, mass 0.05; collision mesh filename=file:///home/albert/rad_ws/install/agbot_full_description/s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 scale=0.004 0.004 0.004; visual mesh filename=file:///home/albert/rad_ws/install/agbot_full_description/s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 scale=0.004 0.004 0.004
- added link elbow_link, mass 0.05; collision cylinder length=0.18 radius=0.015; visual cylinder length=0.18 radius=0.015
- added link forward_drive_arm_link, mass 0.1; collision box size=0.75 0.05 0.005; visual box size=0.75 0.05 0.005
- added link gripper_left_link, mass 0.01; collision mesh filename=file:///home/albert/rad_ws/install/agbot_full_description/s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 scale=0.004 0.004 0.004; visual mesh filename=file:///home/albert/rad_ws/install/agbot_full_description/s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 scale=0.004 0.004 0.004
- added link gripper_right_link, mass 0.01; collision mesh filename=file:///home/albert/rad_ws/install/agbot_full_description/s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 scale=0.004 0.004 0.004; visual mesh filename=file:///home/albert/rad_ws/install/agbot_full_description/s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 scale=0.004 0.004 0.004
- added link horizontal_arm_link, mass 0.1; collision box size=0.555 0.05 0.005; visual box size=0.555 0.05 0.005
- added link roboball_cylinder_link, mass 3.0; collision cylinder length=1.8288 radius=0.2032; visual cylinder length=1.8288 radius=0.2032
- added link wrist_link, mass 0.05; collision cylinder length=0.18 radius=0.015; visual cylinder length=0.09 radius=0.015
- link arm_base_car_link: mass 2.0 -> 0.5
- link arm_base_link: geometry collision mesh filename=file:///home/albert/bcdc_ws/install/agbot_description/share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 scale=0.0015 0.0015 0.002; visual mesh filename=file:///home/albert/bcdc_ws/install/agbot_description/share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 scale=0.0015 0.0015 0.002
- link arm_base_rail_link: mass 2.0 -> 0.5
- link arm_mid_rail_link: mass 2.0 -> 0.5
- link box_four_link: mass 10.0 -> 0.2
- link box_one_link: mass 10.0 -> 0.2
- link box_three_link: mass 10.0 -> 0.2
- link box_two_link: mass 10.0 -> 0.2
Joints:
- joint arm_base_joint: child base_plate -> base_plate_link
- joint arm_camera_optical_joint: child arm_rgb_camera_optical -> arm_rgb_camera_optical_link; parent claw_support -> claw_support_link
- joint arm_rgb_camera_joint: child arm_rgb_camera -> arm_rgb_camera_link; parent arm_rgb_camera_optical -> arm_rgb_camera_optical_link
- joint body_arm_joint: origin xyz=0 0 0.8001 rpy=0 0 1.570796326795 -> xyz=0 -0.1397 0 rpy=0 1.570796326795 1.570796326795; parent base_link -> roboball_cylinder_link
- joint elbow_forearm_joint: child wrist -> wrist_link; parent horizontal_arm -> horizontal_arm_link
- joint elbow_joint: child horizontal_arm -> horizontal_arm_link; parent elbow -> elbow_link
- joint gripper_left_joint: child gripper_left -> gripper_left_link; origin xyz=0.040 -0.014 0.083 -> xyz=0.042 -0.015 0.083; parent claw_support -> claw_support_link
- joint gripper_right_joint: child gripper_right -> gripper_right_link; origin xyz=-0.035 -0.014 0.083 -> xyz=-0.037 -0.015 0.083; parent claw_support -> claw_support_link
- joint robo_cylinder_joint: child roboball_cylinder -> roboball_cylinder_link
- joint shoulder_elbow_joint: child elbow -> elbow_link; parent forward_drive_arm -> forward_drive_arm_link
- joint shoulder_joint: child forward_drive_arm -> forward_drive_arm_link; parent base_plate -> base_plate_link
- joint wrist_joint: child claw_support -> claw_support_link; parent wrist -> wrist_link

File: install/agbot_full_description/share/agbot_full_description/urdf/agbot_full.xacro (robot description, xacro)
@@ -186,4 +186,72 @@
     </link>
     <!-- Robot Arm -->
+     <link name = "roboball_cylinder_link">
+        <visual>
+            <geometry>
+                <cylinder length = "${robo_cylinder_length}" radius = "${robo_cylinder_radius}" />
+            </geometry>
+            <origin xyz = "0 0 0" rpy = "0 0 0" />
+            <material name = "ClearGrey" />
+        </visual>
+        <collision>
+            <geometry>
+                <cylinder length = "${robo_cylinder_length}" radius = "${robo_cylinder_radius}" />
+            </geometry>
+            <origin xyz = "0 0 0" rpy = "0 0 0" />
+        </collision>
+        <xacro:cylinder_inertia m = "3.0" r = "${robo_cylinder_radius}" h = "${robo_cylinder_length}"
+                                xyz = "0 0 0" rpy = "0 0 0"/>
+    </link>
+    <link name="arm_base_rail_link">
+        <visual>
+            <geometry>
+                <box size="${arm_base_rail_length} ${arm_base_rail_width} ${arm_base_rail_height}"/>
+            </geometry>
+            <origin xyz="0 0 0" rpy="0 0 0"/>
+            <material name="white"/>
+        </visual>
+        <collision>
+            <geometry>
+                <box size="${arm_base_rail_length} ${arm_base_rail_width} ${arm_base_rail_height}"/>
+            </geometry>
+            <origin xyz="0 0 0" rpy="0 0 0"/>
+        </collision>
+        <xacro:box_inertia m="0.5" l="${arm_base_rail_length}" w="${arm_base_rail_width}" h="${arm_base_rail_height}"
+                        xyz = "0 0 ${arm_base_rail_height/2}" rpy="0 0 0" />
+    </link>
+    <link name="arm_mid_rail_link">
+        <visual>
+            <geometry>
+                <box size="${arm_base_rail_length} ${arm_base_rail_width} ${arm_base_rail_height}"/>
+            </geometry>
+            <origin xyz="0 0 0" rpy="0 0 0"/>
+            <material name="black"/>
+        </visual>
+        <collision>
+            <geometry>
+                 <box size="${arm_base_rail_length} ${arm_base_rail_width} ${arm_base_rail_height}"/>
+            </geometry>
+            <origin xyz="0 0 0" rpy="0 0 0"/>
+        </collision>
+        <xacro:box_inertia m="0.5" l="${arm_base_rail_length}" w="${arm_base_rail_width}" h="${arm_base_rail_height}"
+                           xyz = "0 0 ${arm_base_rail_height/2}" rpy="0 0 0" />
+    </link>
+    <link name="arm_base_car_link">
+        <visual>
+            <geometry>
+                <box size="${arm_base_car_length} ${arm_base_car_width} ${arm_base_car_height}"/>
+            </geometry>
+            <origin xyz="0 0 ${arm_base_car_height/2}" rpy="0 0 0"/>
+            <material name="white"/>
+        </visual>
+        <collision>
+            <geometry>
+                <box size="${arm_base_car_length} ${arm_base_car_width} ${arm_base_car_height}"/>
+            </geometry>
+            <origin xyz="0 0 ${arm_base_car_height/2}" rpy="0 0 0"/>
+        </collision>
+        <xacro:box_inertia m="0.5" l="${arm_base_car_length}" w="${arm_base_car_width}" h="${arm_base_car_height}"
+                           xyz = "0 0 ${arm_base_car_height/2}" rpy="0 0 0" />
+    </link>
     <xacro:macro name="box_link" params="prefix" >
         <link name="box_${prefix}_link">
@@ -201,5 +269,5 @@
                 <origin xyz="0 0 ${box_height/2}" rpy="0 0 0"/>
             </collision>
-            <xacro:box_inertia m="10.0" l="${box_length}" w="${box_width}" h="${box_height}"
+            <xacro:box_inertia m="0.2" l="${box_length}" w="${box_width}" h="${box_height}"
                                xyz = "0 0 ${box_height/2}" rpy="0 0 0" />
         </link>
@@ -209,72 +277,4 @@
     <xacro:box_link prefix="three" />
     <xacro:box_link prefix="four" />
-    <link name = "roboball_cylinder">
-        <visual>
-            <geometry>
-                <cylinder length = "${robo_cylinder_length}" radius = "${robo_cylinder_radius}" />
-            </geometry>
-            <origin xyz = "0 0 0" rpy = "0 0 0" />
-            <material name = "ClearGrey" />
-        </visual>
-        <collision>
-            <geometry>
-                <cylinder length = "${robo_cylinder_length}" radius = "${robo_cylinder_radius}" />
-            </geometry>
-            <origin xyz = "0 0 0" rpy = "0 0 0" />
-        </collision>
-        <xacro:cylinder_inertia m = "0.01" r = "${robo_cylinder_radius}" h = "${robo_cylinder_length}"
-                                xyz = "0 0 0" rpy = "0 0 0"/>
-    </link>
-    <link name="arm_base_rail_link">
-        <visual>
-            <geometry>
-                <box size="${arm_base_rail_length} ${arm_base_rail_width} ${arm_base_rail_height}"/>
-            </geometry>
-            <origin xyz="0 0 0" rpy="0 0 0"/>
-            <material name="white"/>
-        </visual>
-        <collision>
-            <geometry>
-                <box size="${arm_base_rail_length} ${arm_base_rail_width} ${arm_base_rail_height}"/>
-            </geometry>
-            <origin xyz="0 0 0" rpy="0 0 0"/>
-        </collision>
-        <xacro:box_inertia m="2.0" l="${arm_base_rail_length}" w="${arm_base_rail_width}" h="${arm_base_rail_height}"
-                        xyz = "0 0 ${arm_base_rail_height/2}" rpy="0 0 0" />
-    </link>
-    <link name="arm_mid_rail_link">
-        <visual>
-            <geometry>
-                <box size="${arm_base_rail_length} ${arm_base_rail_width} ${arm_base_rail_height}"/>
-            </geometry>
-            <origin xyz="0 0 0" rpy="0 0 0"/>
-            <material name="black"/>
-        </visual>
-        <collision>
-            <geometry>
-                 <box size="${arm_base_rail_length} ${arm_base_rail_width} ${arm_base_rail_height}"/>
-            </geometry>
-            <origin xyz="0 0 0" rpy="0 0 0"/>
-        </collision>
-        <xacro:box_inertia m="2.0" l="${arm_base_rail_length}" w="${arm_base_rail_width}" h="${arm_base_rail_height}"
-                           xyz = "0 0 ${arm_base_rail_height/2}" rpy="0 0 0" />
-    </link>
-    <link name="arm_base_car_link">
-        <visual>
-            <geometry>
-                <box size="${arm_base_car_length} ${arm_base_car_width} ${arm_base_car_height}"/>
-            </geometry>
-            <origin xyz="0 0 ${arm_base_car_height/2}" rpy="0 0 0"/>
-            <material name="white"/>
-        </visual>
-        <collision>
-            <geometry>
-                <box size="${arm_base_car_length} ${arm_base_car_width} ${arm_base_car_height}"/>
-            </geometry>
-            <origin xyz="0 0 ${arm_base_car_height/2}" rpy="0 0 0"/>
-        </collision>
-        <xacro:box_inertia m="2.0" l="${arm_base_car_length}" w="${arm_base_car_width}" h="${arm_base_car_height}"
-                           xyz = "0 0 ${arm_base_car_height/2}" rpy="0 0 0" />
-    </link>
     <link name="arm_base_link">
         <xacro:default_inertia mass="1.0"/>
@@ -293,5 +293,5 @@
         </collision>
     </link>
-    <link name="base_plate">
+    <link name="base_plate_link">
         <xacro:default_inertia mass="0.1"/>
          <visual>
@@ -309,5 +309,5 @@
         </collision>
     </link>
-    <link name="forward_drive_arm">
+    <link name="forward_drive_arm_link">
         <xacro:default_inertia mass="0.1"/>
         <visual>
@@ -325,5 +325,5 @@
         </collision>
     </link>
-    <link name = "elbow">
+    <link name = "elbow_link">
         <visual>
             <origin xyz="0 0 0" rpy="0 ${PI / 2} 0"/>
@@ -342,5 +342,5 @@
                                 xyz = "0 0 0" rpy = "0 0 0"/>
     </link>
-    <link name="horizontal_arm">
+    <link name="horizontal_arm_link">
         <xacro:default_inertia mass="0.1"/>
         <visual>
@@ -358,5 +358,5 @@
         </collision>
     </link>
-    <link name = "wrist">
+    <link name = "wrist_link">
         <visual>
             <origin xyz="0 0 0" rpy="0 ${PI / 2} 0"/>
@@ -375,5 +375,5 @@
                                 xyz = "0 0 0" rpy = "0 0 0"/>
     </link>
-    <link name="claw_support">
+    <link name="claw_support_link">
         <xacro:default_inertia mass="0.05"/>
         <visual>
@@ -391,5 +391,5 @@
         </collision>
     </link>
-    <link name="gripper_right">
+    <link name="gripper_right_link">
         <xacro:default_inertia mass="0.01"/>
         <visual>
@@ -407,5 +407,5 @@
         </collision>
     </link>
-    <link name="gripper_left">
+    <link name="gripper_left_link">
         <xacro:default_inertia mass="0.01"/>
         <visual>
@@ -423,7 +423,7 @@
         </collision>
     </link>
-    <link name="arm_rgb_camera_optical" >
-    </link>
-    <link name="arm_rgb_camera">
+    <link name="arm_rgb_camera_optical_link" >
+    </link>
+    <link name="arm_rgb_camera_link">
         <xacro:default_inertia mass="0.001"/>
         <visual>
@@ -488,11 +488,11 @@
     <joint name = "robo_cylinder_joint" type = "fixed">
         <parent link = "base_link"/>
-        <child link="roboball_cylinder" />
+        <child link="roboball_cylinder_link" />
         <origin xyz = "0 0 ${base_height + robo_cylinder_radius}" rpy = "${PI/2} 0 0" />
      </joint>
      <joint name = "body_arm_joint" type = "fixed">
-        <parent link = "base_link"/>
+        <parent link="roboball_cylinder_link" />
         <child link="arm_base_rail_link" />
-        <origin xyz = "0 0 ${base_height + (3*arm_base_rail_height)}" rpy = "0 0 ${PI/2}" />
+        <origin xyz = "0 -${robo_cylinder_radius - (5*arm_base_rail_height)} 0" rpy = "0 ${PI/2} ${PI/2}" />
      </joint>
      <joint name = "base_rail_to_ mid_rail_joint" type = "prismatic">
@@ -536,5 +536,5 @@
     <joint name ="arm_base_joint" type="revolute">
         <parent link="arm_base_link"/>
-        <child link = "base_plate"/>
+        <child link = "base_plate_link"/>
         <origin xyz="0 0 0.07"/>
         <axis xyz="0 0 1"/>
@@ -543,6 +543,6 @@
     </joint>
     <joint name="shoulder_joint" type="revolute">
-        <parent link="base_plate"/>
-        <child link="forward_drive_arm"/>
+        <parent link="base_plate_link"/>
+        <child link="forward_drive_arm_link"/>
         <origin xyz="0 0 0.075" rpy="-${PI/2} 0 0"/>
         <axis xyz="1 0 0"/>
@@ -550,11 +550,11 @@
     </joint>
     <joint name = "shoulder_elbow_joint" type = "fixed">
-        <parent link = "forward_drive_arm"/>
-        <child link = "elbow"/>
+        <parent link = "forward_drive_arm_link"/>
+        <child link = "elbow_link"/>
         <origin xyz = "${(forward_drive_arm_width / 1.5) + 0.02} 0 ${forward_drive_arm_length}" rpy = "0 0 0"/>
     </joint>
     <joint name="elbow_joint" type="revolute">
-        <parent link="elbow"/>
-        <child link="horizontal_arm"/>
+        <parent link="elbow_link"/>
+        <child link="horizontal_arm_link"/>
         <origin xyz="${cylinder_length/4} 0 0" rpy="-${PI} 0 0"/>
         <axis xyz="1 0 0"/>
@@ -562,11 +562,11 @@
     </joint>
     <joint name = "elbow_forearm_joint" type = "fixed">
-        <parent link = "horizontal_arm"/>
-        <child link = "wrist"/>
+        <parent link = "horizontal_arm_link"/>
+        <child link = "wrist_link"/>
         <origin xyz = "0 0 ${horizontal_arm_length}" rpy = "0 0 0"/>
     </joint>
     <joint name="wrist_joint" type="revolute">
-        <parent link="wrist"/>
-        <child link="claw_support"/>
+        <parent link="wrist_link"/>
+        <child link="claw_support_link"/>
         <origin xyz="0 0 0" />
         <axis xyz="1 0 0"/>
@@ -574,7 +574,7 @@
     </joint>
     <joint name="gripper_right_joint" type="revolute">
-        <parent link="claw_support"/>
-        <child link="gripper_right"/>
-        <origin xyz="-0.035 -0.014 0.083"/>
+        <parent link="claw_support_link"/>
+        <child link="gripper_right_link"/>
+        <origin xyz="-0.037 -0.015 0.083"/>
         <axis xyz="0 1 0"/>
         <limit lower="-${PI / 2}" upper="0.0" effort="${effort}" velocity="${velocity}"/>
@@ -582,18 +582,18 @@
     <joint name="gripper_left_joint" type="revolute">
         <mimic joint="gripper_right_joint" multiplier="-1"/>
-        <parent link="claw_support"/>
-        <child link="gripper_left"/>
-        <origin xyz="0.040 -0.014 0.083"/>
+        <parent link="claw_support_link"/>
+        <child link="gripper_left_link"/>
+        <origin xyz="0.042 -0.015 0.083"/>
         <axis xyz="0 1 0"/>
         <limit lower="0.0" upper="${PI / 2}" effort="${effort}" velocity="${velocity}"/>
     </joint>
     <joint name="arm_camera_optical_joint" type="fixed">
-        <parent link="claw_support"/>
-        <child link="arm_rgb_camera_optical"/>
+        <parent link="claw_support_link"/>
+        <child link="arm_rgb_camera_optical_link"/>
         <origin xyz = "0 .10 0.085" rpy = "0 0 0" />
     </joint>
     <joint name = "arm_rgb_camera_joint" type = "fixed" >
-        <parent link = "arm_rgb_camera_optical" />
-        <child link = "arm_rgb_camera" />
+        <parent link = "arm_rgb_camera_optical_link" />
+        <child link = "arm_rgb_camera_link" />
         <origin xyz="0 0 0.03" rpy="0 -${PI/2} 0"/>
     </joint>

File: install/agbot_full_description/share/agbot_full_description/urdf/agbot_full_gazebo.xacro (robot description, xacro)
@@ -105,27 +105,32 @@
     <gazebo reference="base_link">
         <material>Gazebo/White</material>
-     </gazebo>
-     <gazebo reference="left_wheel_link">
-        <material>Gazebo/Black</material>
-        <mu1 value="0.8"/>
-        <mu2 value="0.8"/>
-     </gazebo>
-     <gazebo reference="right_wheel_link">
-        <material>Gazebo/Black</material>
-        <mu1 value="0.8"/>
-        <mu2 value="0.8"/>
-     </gazebo>
-     <gazebo reference="caster_wheel_link">
-        <material>Gazebo/Yellow</material>
-        <mu1 value="0.0001"/>
-        <mu2 value="0.0001"/>
-     </gazebo>
-     <gazebo reference="rgb_camera">
-        <material>Gazebo/DarkGrey</material>
-     </gazebo>
-     <gazebo reference="mast_link">
-        <material>Gazebo/Purple</material>
-     </gazebo>
+    </gazebo>
+    <gazebo reference="left_wheel_link">
+      <material>Gazebo/Black</material>
+      <mu1 value="0.8"/>
+      <mu2 value="0.8"/>
+    </gazebo>
+    <gazebo reference="right_wheel_link">
+      <material>Gazebo/Black</material>
+      <mu1 value="0.8"/>
+      <mu2 value="0.8"/>
+    </gazebo>
+    <gazebo reference="caster_wheel_link">
+      <material>Gazebo/Yellow</material>
+      <mu1 value="0.0001"/>
+      <mu2 value="0.0001"/>
+    </gazebo>
+    <gazebo reference="rgb_camera">
+      <material>Gazebo/DarkGrey</material>
+    </gazebo>
+    <gazebo reference="mast_link">
+      <material>Gazebo/Purple</material>
+    </gazebo>
     <!-- Robot Arm -->
+    <gazebo reference = "roboball_cylinder_link">
+      <material>Gazebo/GreyTransparent</material>
+      <mu1>30.0</mu1>
+      <mu2>30.0</mu2>
+    </gazebo>
     <gazebo reference="arm_base_rail_link">
         <material>Gazebo/White</material>
@@ -149,30 +154,30 @@
         <minDepth>0.001</minDepth>
     </gazebo>
-     <gazebo reference="arm_base_link">
-        <material>Gazebo/Blue</material>
-      </gazebo>
-      <gazebo reference="base_plate">
-        <material>Gazebo/Red</material>
-      </gazebo>
-      <gazebo reference="forward_drive_arm">
-        <material>Gazebo/Yellow</material>
-      </gazebo>
-      <gazebo reference="elbow">
-        <material>Gazebo/White</material>
-      </gazebo>
-      <gazebo reference="horizontal_arm">
-        <material>Gazebo/Green</material>
-      </gazebo>
-      <gazebo reference="claw_support">
-        <material>Gazebo/Yellow</material>
-      </gazebo>
-      <gazebo reference="gripper_right">
-        <material>Gazebo/Purple</material>
-      </gazebo>
-      <gazebo reference="gripper_left">
-        <material>Gazebo/Purple</material>
-      </gazebo>
-      <gazebo reference="arm_rgb_camera">
-        <material>Gazebo/Blue</material>
-      </gazebo>
+    <gazebo reference="arm_base_link">
+      <material>Gazebo/Blue</material>
+    </gazebo>
+    <gazebo reference="base_plate_link">
+      <material>Gazebo/Red</material>
+    </gazebo>
+    <gazebo reference="forward_drive_arm_link">
+      <material>Gazebo/Yellow</material>
+    </gazebo>
+    <gazebo reference="elbow_link">
+      <material>Gazebo/White</material>
+    </gazebo>
+    <gazebo reference="horizontal_arm_link">
+      <material>Gazebo/Green</material>
+    </gazebo>
+    <gazebo reference="claw_support_link">
+      <material>Gazebo/Yellow</material>
+    </gazebo>
+    <gazebo reference="gripper_right_link">
+      <material>Gazebo/Purple</material>
+    </gazebo>
+    <gazebo reference="gripper_left_link">
+      <material>Gazebo/Purple</material>
+    </gazebo>
+    <gazebo reference="arm_rgb_camera_link">
+      <material>Gazebo/Blue</material>
+    </gazebo>
 </robot>
