Commit message: Cleanup Update

File: install/agbot_full_description/share/agbot_full_description/urdf/agbot_full_ros2_control.xacro (robot description, xacro)
@@ -22,19 +22,15 @@
         <joint name="base_rail_to_ mid_rail_joint">
             <command_interface name="position">
-                <param name="min">0</param>
+                <param name="min">-0.1</param>
                 <param name="max">${((arm_base_rail_length / 2) + (arm_base_rail_length / 4))/2}</param>
             </command_interface>
             <state_interface name="position"/>
-            <state_interface name="velocity"/>
-            <state_interface name="effort"/>
         </joint>
         <joint name="mid_rail_to_arm_car_joint">
             <command_interface name="position">
-                <param name="min">0</param>
+                <param name="min">-0.1</param>
                 <param name="max">$${(arm_base_rail_length / 2) + (arm_base_rail_length / 4)}</param>
             </command_interface>
             <state_interface name="position"/>
-            <state_interface name="velocity"/>
-            <state_interface name="effort"/>
         </joint>
         <joint name="arm_base_joint">
@@ -68,8 +64,10 @@
         <joint name="gripper_right_joint">
             <command_interface name="position">
-                <param name="min">-${PI/2}</param>
-                <param name="max">0</param>
+            <!-- <command_interface name="effort"> -->
+                <param name="min">-${(PI/2)+.01}</param>
+                <param name="max">0.01</param>
             </command_interface>
             <state_interface name="position"/>
+            <!-- <state_interface name="effort"/> -->
         </joint>
         <joint name="gripper_left_joint">
@@ -77,5 +75,6 @@
             <param name="multiplier">-1</param>
             <command_interface name="position">
-                <param name="min">0</param>
+            <!-- <command_interface name="effort"> -->
+                <param name="min">-0.01</param>
                 <param name="max">${PI/2}</param>
             </command_interface>

File: install/agbot_full_moveit/share/agbot_full_moveit/config/agbot_full.urdf (robot description, URDF)
Before this commit: robot agbot_full, 28 links, 27 joints
Links:
- removed link arm_rgb_camera
- removed link arm_rgb_camera_optical
- removed link base_plate
- removed link claw_support
- removed link elbow
- removed link forward_drive_arm
- removed link gripper_left
- removed link gripper_right
- removed link horizontal_arm
- removed link roboball_cylinder
- removed link wrist
- added link arm_rgb_camera_link, mass 0.001; collision mesh filename=file:///home/albert/rad_ws/install/agbot_full_description/s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 scale=0.002 0.002 0.002; visual mesh filename=file:///home/albert/rad_ws/install/agbot_full_description/s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 scale=0.002 0.002 0.002
- added link arm_rgb_camera_optical_link
- added link base_plate_link, mass 0.1; collision mesh filename=file:///home/albert/bcdc_ws/install/agbot_description/share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 scale=0.0015 0.0015 0.002; visual mesh filename=file:///home/albert/bcdc_ws/install/agbot_description/share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 scale=0.0015 0.0015 0.002
- added link claw_support_link, mass 0.05; collision mesh filename=file:///home/albert/rad_ws/install/agbot_full_description/s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 scale=0.004 0.004 0.004; visual mesh filename=file:///home/albert/rad_ws/install/agbot_full_description/s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 scale=0.004 0.004 0.004
- added link elbow_link, mass 0.05; collision cylinder length=0.18 radius=0.015; visual cylinder length=0.18 radius=0.015
- added link forward_drive_arm_link, mass 0.1; collision box size=0.75 0.05 0.005; visual box size=0.75 0.05 0.005
- added link gripper_left_link, mass 0.01; collision mesh filename=file:///home/albert/rad_ws/install/agbot_full_description/s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 scale=0.004 0.004 0.004; visual mesh filename=file:///home/albert/rad_ws/install/agbot_full_description/s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 scale=0.004 0.004 0.004
- added link gripper_right_link, mass 0.01; collision mesh filename=file:///home/albert/rad_ws/install/agbot_full_description/s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 scale=0.004 0.004 0.004; visual mesh filename=file:///home/albert/rad_ws/install/agbot_full_description/s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 scale=0.004 0.004 0.004
- added link horizontal_arm_link, mass 0.1; collision box size=0.555 0.05 0.005; visual box size=0.555 0.05 0.005
- added link roboball_cylinder_link, mass 3.0; collision cylinder length=1.8288 radius=0.2032; visual cylinder length=1.8288 radius=0.2032
- added link wrist_link, mass 0.05; collision cylinder length=0.18 radius=0.015; visual cylinder length=0.09 radius=0.015
- link arm_base_car_link: mass 2.0 -> 0.5
- link arm_base_link: geometry collision mesh filename=file:///home/albert/bcdc_ws/install/agbot_description/share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 scale=0.0015 0.0015 0.002; visual mesh filename=file:///home/albert/bcdc_ws/install/agbot_description/share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 scale=0.0015 0.0015 0.002
- link arm_base_rail_link: mass 2.0 -> 0.5
- link arm_mid_rail_link: mass 2.0 -> 0.5
- link box_four_link: mass 10.0 -> 0.2
- link box_one_link: mass 10.0 -> 0.2
- link box_three_link: mass 10.0 -> 0.2
- link box_two_link: mass 10.0 -> 0.2
Joints:
- joint arm_base_joint: child base_plate -> base_plate_link
- joint arm_camera_optical_joint: child arm_rgb_camera_optical -> arm_rgb_camera_optical_link; parent claw_support -> claw_support_link
- joint arm_rgb_camera_joint: child arm_rgb_camera -> arm_rgb_camera_link; parent arm_rgb_camera_optical -> arm_rgb_camera_optical_link
- joint body_arm_joint: origin xyz=0 0 0.8001 rpy=0 0 1.570796326795 -> xyz=0 -0.1397 0 rpy=0 1.570796326795 1.570796326795; parent base_link -> roboball_cylinder_link
- joint elbow_forearm_joint: child wrist -> wrist_link; parent horizontal_arm -> horizontal_arm_link
- joint elbow_joint: child horizontal_arm -> horizontal_arm_link; parent elbow -> elbow_link
- joint gripper_left_joint: child gripper_left -> gripper_left_link; origin xyz=0.040 -0.014 0.083 -> xyz=0.042 -0.015 0.083; parent claw_support -> claw_support_link
- joint gripper_right_joint: child gripper_right -> gripper_right_link; origin xyz=-0.035 -0.014 0.083 -> xyz=-0.037 -0.015 0.083; parent claw_support -> claw_support_link
- joint robo_cylinder_joint: child roboball_cylinder -> roboball_cylinder_link
- joint shoulder_elbow_joint: child elbow -> elbow_link; parent forward_drive_arm -> forward_drive_arm_link
- joint shoulder_joint: child forward_drive_arm -> forward_drive_arm_link; parent base_plate -> base_plate_link
- joint wrist_joint: child claw_support -> claw_support_link; parent wrist -> wrist_link

Commit message: Update 04OCT24

File: install/agbot_full_description/share/agbot_full_description/urdf/agbot_full.urdf (robot description, URDF)
Before this commit: robot agbot_full, 28 links, 27 joints
Links:
- removed link laser_frame
- removed link rgb_camera
- removed link rgb_camera_optical
- added link laser_frame_link
- added link laser_link, mass 0.1; collision cylinder length=0.1 radius=0.025; visual cylinder length=0.1 radius=0.025
- added link rgb_camera_link, mass 0.001; collision mesh filename=file:///home/albert/rad_ws/install/agbot_full_description/s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 scale=0.0025 0.0025 0.0025; visual mesh filename=file:///home/albert/rad_ws/install/agbot_full_description/s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 scale=0.0025 0.0025 0.0025
- added link rgb_camera_optical_link
- link caster_wheel_link: mass 0.2 -> 2.0
- link left_wheel_link: mass 1.0 -> 3.0
- link mast_link: geometry collision box size=0.05 0.05 0.15; visual box size=0.05 0.05 0.15
- link right_wheel_link: mass 1.0 -> 3.0
Joints:
- added joint laser_frame_joint: type fixed, parent mast_link, child laser_frame_link, origin xyz=0 0 0.15 rpy=0 0 0
- joint base_mast_joint: origin xyz=0.9394 0 0.5715 rpy=0 0 0 -> xyz=0.8644 0 0.762 rpy=0 0 0
- joint camera_optical_joint: child rgb_camera_optical -> rgb_camera_optical_link
- joint laser_joint: child laser_frame -> laser_link; parent mast_link -> laser_frame_link
- joint rgb_camera_joint: child rgb_camera -> rgb_camera_link; parent rgb_camera_optical -> rgb_camera_optical_link

File: install/agbot_full_description/share/agbot_full_description/urdf/agbot_full.xacro (robot description, xacro)
@@ -23,5 +23,5 @@
     <xacro:property name="mast_length" value="0.05" />
     <xacro:property name="mast_width" value="0.05" />
-    <xacro:property name="mast_height" value="0.03" />
+    <xacro:property name="mast_height" value="0.15" />
     <xacro:property name="caster_radius" value="0.162" />
     <xacro:property name = "forward_drive_arm_length" value = "0.75" />
@@ -33,4 +33,6 @@
     <xacro:property name = "cylinder_radius" value = "0.015" />
     <xacro:property name = "cylinder_length" value = "0.18" />
+    <xacro:property name = "laser_radius" value = "0.025" />
+    <xacro:property name = "laser_length" value = "0.10" />
     <xacro:property name = "robo_cylinder_radius" value = "0.2032" />
     <xacro:property name = "robo_cylinder_length" value = "1.8288" />
@@ -66,12 +68,15 @@
     <xacro:macro name="prismatic_transmission" params="name">
         <transmission name="${name}_prismatic_transmission">
-            <type>transmission_interface/SimpleTransmission</type>
+            <!-- <type>transmission_interface/SimpleTransmission</type> -->
+            <type>"velocity_controllers/JointPositionController"</type>
             <!-- <plugin>hardware_interface/VelocityJointInterface</plugin> -->
             <joint name="${name}">
-                <hardwareInterface>hardware_interface/PositionJointInterface</hardwareInterface>
+                <hardwareInterface>hardware_interface/VelocityJointInterface</hardwareInterface>
+                <!-- <hardwareInterface>hardware_interface/PositionJointInterface</hardwareInterface> -->
             </joint>
             <actuator name="${name}_motor">
-                <hardwareInterface>hardware_interface/PositionJointInterface</hardwareInterface>
-                <mechanicalReduction>1</mechanicalReduction>
+                <hardwareInterface>hardware_interface/VelocityJointInterface</hardwareInterface>
+                <!-- <hardwareInterface>hardware_interface/PositionJointInterface</hardwareInterface> -->
+                <mechanicalReduction>1.0</mechanicalReduction>
             </actuator>
         </transmission>
@@ -111,5 +116,5 @@
             <origin xyz = "0 0 0" rpy = "0 0 0" />
         </collision>
-        <xacro:wheel_inertia m="1.0" r = "${wheel_radius}" h = "${wheel_length}"
+        <xacro:wheel_inertia m="3.0" r = "${wheel_radius}" h = "${wheel_length}"
                              xyz = "0 0 0" rpy = "${Pi/2.0} -${Pi/2.0} 0" />
     </link>
@@ -128,5 +133,5 @@
             <origin xyz = "0 0 0" rpy = "0 0 0" />
         </collision>
-        <xacro:wheel_inertia m="1.0" r = "${wheel_radius}" h = "${wheel_length}"
+        <xacro:wheel_inertia m="3.0" r = "${wheel_radius}" h = "${wheel_length}"
                              xyz = "0 0 0" rpy = "${Pi/2.0} -${Pi/2.0} 0" />
     </link>
@@ -145,10 +150,10 @@
             <origin xyx = "${base_length / 3} 0 ${caster_radius}" rpy = "0 0 0" />
         </collision>
-        <xacro:sphere_inertia m = "0.2" r = "${caster_radius}"
+        <xacro:sphere_inertia m = "2.0" r = "${caster_radius}"
                             xyz = "${base_length / 3} 0 0" rpy = "0 0 0" />
     </link>
-    <link name="rgb_camera_optical" >
-    </link>
-    <link name="rgb_camera">
+    <link name="rgb_camera_optical_link" >
+    </link>
+    <link name="rgb_camera_link">
         <xacro:default_inertia mass="0.001"/>
         <visual>
@@ -183,5 +188,22 @@
                             xyz = "0 0 0" rpy="0 0 0" />
     </link>
-    <link name="laser_frame">
+    <link name="laser_frame_link">
+    </link>
+    <link name="laser_link">
+        <visual>
+            <geometry>
+                <cylinder length="${laser_length}" radius="${laser_radius}" />
+            </geometry>
+            <origin xyz = "0 0 0" rpy = "0 0 0" />
+            <material name="red"/>
+        </visual>
+        <collision>
+            <geometry>
+                <cylinder length="${laser_length}" radius="${laser_radius}" />
+            </geometry>
+            <origin xyz = "0 0 0" rpy = "0 0 0" />
+        </collision>
+        <xacro:cylinder_inertia m="0.1" r="${laser_radius}" h="${laser_length}"
+                                 xyz="0 0 0" rpy="0 0 0"/>
     </link>
     <!-- Robot Arm -->
@@ -451,5 +473,5 @@
         <parent link="base_link" />
         <child link="right_wheel_link" />
-        <origin xyz="-${base_length / 4.0} -${(base_width + wheel_length) / 2.0} ${wheel_radius}" rpy="0 0 0" />
+        <origin xyz="-${base_length / 4.0} -${(base_width + (5*wheel_length)) / 2.0} ${wheel_radius}" rpy="0 0 0" />
         <axis xyz="0 1 0" />
     </joint>
@@ -457,5 +479,5 @@
         <parent link="base_link" />
         <child link="left_wheel_link" />
-        <origin xyz="-${base_length / 4.0} ${(base_width + wheel_length) / 2.0} ${wheel_radius}" rpy="0 0 0" />
+        <origin xyz="-${base_length / 4.0} ${(base_width + (5*wheel_length)) / 2.0} ${wheel_radius}" rpy="0 0 0" />
         <axis xyz="0 1 0" />
     </joint>
@@ -467,10 +489,10 @@
     <joint name="camera_optical_joint" type="fixed">
         <parent link="base_link"/>
-        <child link="rgb_camera_optical"/>
+        <child link="rgb_camera_optical_link"/>
         <origin xyz = "${base_length/2} 0 ${base_height-(base_height/10)}" rpy = "0 0 0" />
     </joint>
     <joint name = "rgb_camera_joint" type = "fixed" >
-        <parent link = "rgb_camera_optical" />
-        <child link = "rgb_camera" />
+        <parent link = "rgb_camera_optical_link" />
+        <child link = "rgb_camera_link" />
         <origin xyz="0 0 0" rpy="0 0 0"/>
     </joint>
@@ -478,9 +500,14 @@
         <parent link = "base_link" />
         <child link = "mast_link" />
-        <origin xyz="${((base_length / 2) + (mast_length / 2))} 0 ${3 * base_height / 4}" rpy="0 0 0"/>
+        <origin xyz="${((base_length / 2) - mast_length)} 0 ${base_height}" rpy="0 0 0"/>
+    </joint>
+    <joint name="laser_frame_joint" type="fixed">
+        <parent link="mast_link"/>
+        <child link="laser_frame_link"/>
+        <origin xyz="0 0 ${mast_height}" rpy="0 0 0"/>
     </joint>
     <joint name="laser_joint" type="fixed">
-        <parent link="mast_link"/>
-        <child link="laser_frame"/>
+        <parent link="laser_frame_link"/>
+        <child link="laser_link"/>
         <origin xyz="0 0 0" rpy="0 0 0"/>
     </joint>
@@ -490,36 +517,36 @@
         <child link="roboball_cylinder_link" />
         <origin xyz = "0 0 ${base_height + robo_cylinder_radius}" rpy = "${PI/2} 0 0" />
-     </joint>
-     <joint name = "body_arm_joint" type = "fixed">
-        <parent link="roboball_cylinder_link" />
-        <child link="arm_base_rail_link" />
-        <origin xyz = "0 -${robo_cylinder_radius - (5*arm_base_rail_height)} 0" rpy = "0 ${PI/2} ${PI/2}" />
-     </joint>
-     <joint name = "base_rail_to_ mid_rail_joint" type = "prismatic">
-        <parent link = "arm_base_rail_link"/>
-        <child link="arm_mid_rail_link" />
-        <origin xyz = "0 0 ${arm_base_rail_height}" rpy = "0 0 0" />
-        <limit lower="0" upper="${((arm_base_rail_length / 2) + (arm_base_rail_length / 4))/2}" effort="100.0" velocity="0.5"/>
-     </joint>
-     <joint name = "box_one_joint" type = "fixed">
-        <parent link = "arm_base_car_link"/>
-        <child link = "box_one_link" />
-        <origin xyz = "-${(arm_base_rail_length / 2) - (box_length / 2)} 0 ${arm_base_rail_height}" rpy = "0 0 0"/>
-     </joint>
-     <joint name = "box_two_joint" type = "fixed">
-        <parent link = "arm_base_car_link"/>
-        <child link = "box_two_link" />
-        <origin xyz = "-${(arm_base_rail_length / 2) - (box_length * 1.5) - 0.05} 0 ${arm_base_rail_height}" rpy = "0 0 0"/>
-     </joint>
-     <joint name = "box_three_joint" type = "fixed">
-        <parent link = "arm_base_car_link"/>
-        <child link = "box_three_link" />
-        <origin xyz = "${(box_length / 2) - 0.05} 0 ${arm_base_rail_height}" rpy = "0 0 0"/>
-     </joint>
-     <joint name = "box_four_joint" type = "fixed">
-        <parent link = "arm_base_car_link"/>
-        <child link = "box_four_link" />
-        <origin xyz = "${box_length *1.5} 0 ${arm_base_rail_height}" rpy = "0 0 0"/>
-     </joint>
+    </joint>
+    <joint name = "body_arm_joint" type = "fixed">
+    <parent link="roboball_cylinder_link" />
+    <child link="arm_base_rail_link" />
+    <origin xyz = "0 -${robo_cylinder_radius - (5*arm_base_rail_height)} 0" rpy = "0 ${PI/2} ${PI/2}" />
+    </joint>
+    <joint name = "base_rail_to_ mid_rail_joint" type = "prismatic">
+    <parent link = "arm_base_rail_link"/>
+    <child link="arm_mid_rail_link" />
+    <origin xyz = "0 0 ${arm_base_rail_height}" rpy = "0 0 0" />
+    <limit lower="0" upper="${((arm_base_rail_length / 2) + (arm_base_rail_length / 4))/2}" effort="100.0" velocity="0.5"/>
+    </joint>
+    <joint name = "box_one_joint" type = "fixed">
+    <parent link = "arm_base_car_link"/>
+    <child link = "box_one_link" />
+    <origin xyz = "-${(arm_base_rail_length / 2) - (box_length / 2)} 0 ${arm_base_rail_height}" rpy = "0 0 0"/>
+    </joint>
+    <joint name = "box_two_joint" type = "fixed">
+    <parent link = "arm_base_car_link"/>
+    <child link = "box_two_link" />
+    <origin xyz = "-${(arm_base_rail_length / 2) - (box_length * 1.5) - 0.05} 0 ${arm_base_rail_height}" rpy = "0 0 0"/>
+    </joint>
+    <joint name = "box_three_joint" type = "fixed">
+    <parent link = "arm_base_car_link"/>
+    <child link = "box_three_link" />
+    <origin xyz = "${(box_length / 2) - 0.05} 0 ${arm_base_rail_height}" rpy = "0 0 0"/>
+    </joint>
+    <joint name = "box_four_joint" type = "fixed">
+    <parent link = "arm_base_car_link"/>
+    <child link = "box_four_link" />
+    <origin xyz = "${box_length *1.5} 0 ${arm_base_rail_height}" rpy = "0 0 0"/>
+    </joint>
     <!-- Robot Arm -->
     <joint name = "mid_rail_to_arm_car_joint" type = "prismatic">

File: install/agbot_full_description/share/agbot_full_description/urdf/agbot_full_gazebo.xacro (robot description, xacro)
@@ -11,5 +11,5 @@
             <left_joint>base_left_wheel_joint</left_joint>
             <right_joint>base_right_wheel_joint</right_joint>
-            <wheel_separation>0.179</wheel_separation>
+            <wheel_separation>1.8288</wheel_separation>
             <wheel_diameter>0.066</wheel_diameter>
             <max_wheel_torque>200.0</max_wheel_torque>
@@ -75,5 +75,5 @@
         </sensor>
       </gazebo>
-      <gazebo reference="laser_frame">
+      <gazebo reference="laser_link">
         <sensor name="laser" type="ray">
             <pose> 0 0 0 0 0 0 </pose>
@@ -87,4 +87,9 @@
                         <max_angle>3.14</max_angle>
                     </horizontal>
+                    <vertical>
+                        <samples>1</samples>
+                        <min_angle>0</min_angle>
+                        <max_angle>0</max_angle>
+                    </vertical>
                 </scan>
                 <range>
@@ -107,10 +112,10 @@
     </gazebo>
     <gazebo reference="left_wheel_link">
-      <material>Gazebo/Black</material>
+      <material>Gazebo/Grey</material>
       <mu1 value="0.8"/>
       <mu2 value="0.8"/>
     </gazebo>
     <gazebo reference="right_wheel_link">
-      <material>Gazebo/Black</material>
+      <material>Gazebo/Grey</material>
       <mu1 value="0.8"/>
       <mu2 value="0.8"/>
@@ -121,9 +126,12 @@
       <mu2 value="0.0001"/>
     </gazebo>
-    <gazebo reference="rgb_camera">
+    <gazebo reference="rgb_camera_link">
       <material>Gazebo/DarkGrey</material>
     </gazebo>
     <gazebo reference="mast_link">
       <material>Gazebo/Purple</material>
+    </gazebo>
+    <gazebo reference="laser_link">
+      <material>Gazebo/Grey</material>
     </gazebo>
     <!-- Robot Arm -->

File: install/agbot_full_description/share/agbot_full_description/urdf/agbot_full_ros2_control.xacro (robot description, xacro)
@@ -26,4 +26,6 @@
             </command_interface>
             <state_interface name="position"/>
+            <!-- <state_interface name="velocity"/>
+            <state_interface name="effort"/> -->
         </joint>
         <joint name="mid_rail_to_arm_car_joint">
@@ -33,4 +35,6 @@
             </command_interface>
             <state_interface name="position"/>
+            <!-- <state_interface name="velocity"/>
+            <state_interface name="effort"/> -->
         </joint>
         <joint name="arm_base_joint">

File: install/agbot_full_moveit_setup/share/agbot_full_moveit_setup/config/agbot_full.ros2_control.xacro (robot description, xacro)
@@ -1,5 +1,5 @@
 <?xml version="1.0"?>
 <robot xmlns:xacro="http://www.ros.org/wiki/xacro">
-    <xacro:macro name="agbot_full_ros2_control" params="name initial_positions_file">
+    <xacro:macro name="agbot_arm_ros2_control" params="name initial_positions_file">
         <xacro:property name="initial_positions" value="${load_yaml(initial_positions_file)['initial_positions']}"/>
         <ros2_control name="${name}" type="system">
